File: Carrier/bme.kicad_sch (KiCad schematic)
At the start: 3 parts, among them U7 BME680

Commit message: Moved lcd screen connector for new screen, corrected LCSC partnumbers
Parts:
- U7: LCSC C125972 -> C42431867
Changed lines of the file:
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@@
 			)
 		)
-		(property "LCSC" "C125972"
+		(property "LCSC" "C42431867"
 			(at 134.62 66.04 0)
 			(effects
