File: M2/flashing.kicad_sch (KiCad schematic)
At the start: 17 parts, among them J2 USB_C_Receptacle_USB2.0_16P, Q2 MMDT2222A, U5 CH340K

Commit message: Moved lcd screen connector for new screen, corrected LCSC partnumbers
Parts:
- R15: LCSC C473048 -> C270365
Changed lines of the file:
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@@
 			)
 		)
-		(property "LCSC" "C473048"
+		(property "LCSC" "C270365"
 			(at 127 35.56 0)
 			(effects
