File: M2/badgeM2Card.kicad_pcb (KiCad board)
At the start: 4 copper layers, 22 x 42 mm, 82 parts, among them IC1 XT25F128FWOIGT-W, IC2 TPS563202DRLR, IC4 TPS563202DRLR, J1 Micro_SD_Card_Det2, J2 USB_C_Receptacle_USB2.0_16P, Q2 MMDT2222A, U2 ESP32-P4NRW16, U5 CH340K, Y1 32KHz, Y2 40MHz

Commit message: Fixed SD det line reconnected to P4
There was an error in the production release. This fixes the problem found after pcb went to production. In case you want to reuse this, with this change the SD card change detection works as intented.
Connections:
- J1 pad 9: GND -> /MCU/SD.DET
- U2 pad 88: GND -> /MCU/SD.DET
Routing:
- net GND: track 110.7 -> 90.2 mm, vias 72 -> 70
- net /MCU/SD.DET: track 0.00 -> 20.5 mm, vias 0 -> 2
Changed lines of the file:
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@@
 	(net 116 "Net-(IC2-BST)")
 	(net 117 "Net-(IC2-SW)")
+	(net 118 "/MCU/SD.DET")
 	(footprint "Resistor_SMD:R_0201_0603Metric"
 		(layer "F.Cu")
@@
 			(size 1.5 0.8)
 			(layers "F.Cu" "F.Mask" "F.Paste")
-			(net 3 "GND")
+			(net 118 "/MCU/SD.DET")
 			(pinfunction "DET_B")
 			(pintype "passive")
@@
 			)
 		)
-		(property "LCSC" "C473048"
+		(property "LCSC" "C270365"
 			(at 0 0 270)
 			(unlocked yes)
@@
 			(size 0.18 0.65)
 			(layers "F.Cu" "F.Paste")
-			(net 3 "GND")
+			(net 118 "/MCU/SD.DET")
 			(pinfunction "GPIO46")
 			(pintype "bidirectional")
@@
 			(net 117 "Net-(IC2-SW)")
 			(pinfunction "SW")
-			(pintype "output")
+			(pintype "power_out")
 		)
 		(pad "3" smd roundrect
@@
 		)
 		(sheetname "/")
-		(sheetfile "P4_M.2_B+M-key.kicad_sch")
+		(sheetfile "badgeM2Card.kicad_sch")
 		(fp_line
 			(start -11 -41.5)
@@
 			(layers "B.Cu" "B.Mask")
 			(net 35 "+3.3V")
-			(pintype "passive")
+			(pintype "power_out")
 			(solder_mask_margin 0.1)
 			(solder_paste_margin 0)
@@
 			(layers "F.Cu" "F.Mask")
 			(net 43 "+5V")
-			(pintype "passive")
+			(pintype "power_out")
 			(solder_mask_margin 0.1)
 			(solder_paste_margin 0)
@@
 		(property ki_fp_filters "LED* LED_SMD:* LED_THT:*")
 		(sheetname "/")
-		(sheetfile "P4_M.2_B+M-key.kicad_sch")
+		(sheetfile "badgeM2Card.kicad_sch")
 		(attr smd)
 		(fp_line
@@
 		(property ki_fp_filters "R_*")
 		(sheetname "/")
-		(sheetfile "P4_M.2_B+M-key.kicad_sch")
+		(sheetfile "badgeM2Card.kicad_sch")
 		(attr smd)
 		(fp_line
@@
 		(property ki_fp_filters "R_*")
 		(sheetname "/")
-		(sheetfile "P4_M.2_B+M-key.kicad_sch")
+		(sheetfile "badgeM2Card.kicad_sch")
 		(attr smd)
 		(fp_line
@@
 			(keep_text_aligned yes)
 		)
-		(gr_text "42,0062"
+		(gr_text "42.0062"
 			(at 165.775 105.0031 90)
 			(layer "F.Fab")
@@
 	)
 	(segment
-		(start 149.7 99.2)
-		(end 151.625 101.125)
-		(width 0.15)
-		(layer "F.Cu")
-		(net 3)
-	)
-	(segment
-		(start 150.15 89.1)
-		(end 150.1 89.05)
-		(width 0.15)
-		(layer "F.Cu")
-		(net 3)
-	)
-	(segment
 		(start 153.2511 124.7536)
 		(end 153.2511 122.9011)
@@
 	)
 	(segment
-		(start 149.7 99.2)
-		(end 149.7 99)
-		(width 0.15)
-		(layer "F.Cu")
-		(net 3)
-	)
-	(segment
 		(start 152.9 103.5)
 		(end 153.1 103.3)
@@
 	)
 	(segment
-		(start 151.625 106.375)
-		(end 151.625 101.125)
-		(width 0.15)
-		(layer "F.Cu")
-		(net 3)
-	)
-	(segment
 		(start 140.3 110.6)
 		(end 141.6 110.6)
@@
 	)
 	(segment
-		(start 151.4 89.1)
-		(end 150.15 89.1)
-		(width 0.15)
-		(layer "F.Cu")
-		(net 3)
-	)
-	(segment
 		(start 150.6 104.68)
 		(end 150.6 103.999)
@@
 	)
 	(via
-		(at 149.7 99)
-		(size 0.45)
-		(drill 0.25)
-		(layers "F.Cu" "B.Cu")
-		(net 3)
-	)
-	(via
 		(at 148.75 122.9)
 		(size 0.45)
@@
 	)
 	(via
-		(at 151.4 89.1)
-		(size 0.45)
-		(drill 0.25)
-		(layers "F.Cu" "B.Cu")
-		(net 3)
-	)
-	(via
 		(at 138 97.2)
 		(size 0.45)
@@
 	)
 	(segment
-		(start 149.7 99)
-		(end 149.7 90.1)
-		(width 0.15)
-		(layer "B.Cu")
-		(net 3)
-	)
-	(segment
 		(start 138.2 111.3)
 		(end 138.2 108.73)
@@
 	)
 	(segment
-		(start 149.7 90.1)
-		(end 150.7 89.1)
-		(width 0.15)
-		(layer "B.Cu")
-		(net 3)
-	)
-	(segment
 		(start 138.2 108.73)
 		(end 138.72 108.21)
@@
 	)
 	(segment
-		(start 150.7 89.1)
-		(end 151.4 89.1)
-		(width 0.15)
-		(layer "B.Cu")
-		(net 3)
-	)
-	(segment
 		(start 143.96 97.99)
 		(end 144.65 97.3)
@@
 		(net 117)
 	)
+	(segment
+		(start 149.7 99.2)
+		(end 151.625 101.125)
+		(width 0.15)
+		(layer "F.Cu")
+		(net 118)
+	)
+	(segment
+		(start 150.15 89.1)
+		(end 150.1 89.05)
+		(width 0.15)
+		(layer "F.Cu")
+		(net 118)
+	)
+	(segment
+		(start 149.7 99.2)
+		(end 149.7 99)
+		(width 0.15)
+		(layer "F.Cu")
+		(net 118)
+	)
+	(segment
+		(start 151.625 106.375)
+		(end 151.625 101.125)
+		(width 0.15)
+		(layer "F.Cu")
+		(net 118)
+	)
+	(segment
+		(start 151.4 89.1)
+		(end 150.15 89.1)
+		(width 0.15)
+		(layer "F.Cu")
+		(net 118)
+	)
+	(via
+		(at 149.7 99)
+		(size 0.45)
+		(drill 0.25)
+		(layers "F.Cu" "B.Cu")
+		(net 118)
+	)
+	(via
+		(at 151.4 89.1)
+		(size 0.45)
+		(drill 0.25)
+		(layers "F.Cu" "B.Cu")
+		(net 118)
+	)
+	(segment
+		(start 149.7 99)
+		(end 149.7 90.1)
+		(width 0.15)
+		(layer "B.Cu")
+		(net 118)
+	)
+	(segment
+		(start 149.7 90.1)
+		(end 150.7 89.1)
+		(width 0.15)
+		(layer "B.Cu")
+		(net 118)
+	)
+	(segment
+		(start 150.7 89.1)
+		(end 151.4 89.1)
+		(width 0.15)
+		(layer "B.Cu")
+		(net 118)
+	)
 	(zone

Commit message: Fix typo in schematic for FLASH
Correction on schematic from FALSH to FLASH. Simple typo correction, nothing more.
Connections:
- net VFALSH renamed VFLASH
Changed lines of the file:
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@@
 	(net 38 "+1.2V")
 	(net 39 "/MCU/GPIO35")
-	(net 40 "VFALSH")
+	(net 40 "VFLASH")
 	(net 41 "VMEM")
 	(net 42 "V{slash}SDMMC")
@@
 			(size 0.65 0.18)
 			(layers "F.Cu" "F.Paste")
-			(net 40 "VFALSH")
+			(net 40 "VFLASH")
 			(pinfunction "VFB1/VO1")
 			(pintype "power_in")
@@
 			(layers "F.Cu" "F.Mask")
 			(roundrect_rratio 0.25)
-			(net 40 "VFALSH")
+			(net 40 "VFLASH")
 			(pintype "passive")
 		)
@@
 			(layers "F.Cu" "F.Mask")
 			(roundrect_rratio 0.25)
-			(net 40 "VFALSH")
+			(net 40 "VFLASH")
 			(pintype "passive")
 		)
@@
 			(layers "F.Cu" "F.Mask" "F.Paste")
 			(roundrect_rratio 0.25)
-			(net 40 "VFALSH")
+			(net 40 "VFLASH")
 			(pinfunction "VCC")
 			(pintype "power_in")
