File: Frontpanel/frontpanel.kicad_sch (KiCad schematic)
At the start: 7 parts

Commit message: Started ripping parts out
Parts:
- removed D1, D2, D3, D4: WS2812B-4020, frontpanel:LED_WS2812B-4020, symbol frontpanel:LED_WS2812B-4020
- removed TP1, TP3, TP6: TestPoint, TestPoint:TestPoint_Pad_D2.0mm, symbol Connector:TestPoint
Connections:
- no-connect marks 1 -> 0
