File: hardware/blackpants.kicad_sch (KiCad schematic)
At the start: 22 parts, among them J1 Conn_01x08, J2 Conn_01x10, J3 Conn_ARM_SWD_TagConnect_TC203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, SW1 SW_Push, U1 STM32F042C6Ux

Commit message: Passing DRC
Parts:
- added C33: 100nF, Capacitor_SMD:C_0402_1005Metric, symbol Device:C_Small
- added R26: 100K, Resistor_SMD:R_0402_1005Metric, symbol Device:R_Small
- added U11: TPSGM7227YUWQ10G, Package_DFN_QFN:UQFN-10_1.4x1.8mm_P0.4mm, symbol Interface_USB:FSUSB42MUX
- JP1, JP2, JP3: footprint (none) -> Jumper:SolderJumper-2_P1.3mm_Bridged_Pad1.0x1.5mm
- SW1: footprint (none) -> Button_Switch_SMD:SW_Push_1P1T_NO_CK_KSC7xxJ
Connections:
- net USART1_RX is gone; now on net USART_RX: JP3.2 (B)
- net +3V3: now also C33.1, R26.1, U11.9 (VCC)
- net COL_4: now also U1.38 (PA15); no longer U1.30 (PA9)
- net GND: now also C33.2, U11.3 (GND), U11.8 (~{OE})
- net USB3.D+: now also U11.5 (HSD1+); no longer U1.33 (PA12)
- net USB3.D-: now also U11.4 (HSD1-); no longer U1.32 (PA11)
- net USB_DET: now reaches U1.2 (PC13)
- net USB_CS: now reaches U1.3 (PC14)
- net USB_CS: now also R26.2, U11.10 (SEL)
- net USART_RX: now reaches U1.31 (PA10)
- net DSI Bridge and Backlight/BL_PWM: now reaches U1.39 (PB3)
- net USART1_TX renamed USART_TX
- net USART_TX: now also U1.30 (PA9)
- new net USB.D+: U11.7 (HSD2+)
- new net USB.D-: U11.6 (HSD2-)
- new net USBSTM.D+: U1.33 (PA12), U11.1 (D+)
- new net USBSTM.D-: U1.32 (PA11), U11.2 (D-)
Other:
- sheet DSI Bridge renamed DSI Bridge and Backlight
- sheet DSI Bridge and Backlight ports: added BL_PWM; removed none
- sheet USB ports: added HS_IND, USB_DET; removed none

Commit message: R0.1 candidate
Parts:
- added S1: Logo_Open_Hardware_Large, Symbol:OSHW-Logo2_24.3x20mm_SilkScreen, symbol Graphic:Logo_Open_Hardware_Large
- C10, C11, C33, C6, C7, C8, C9: LCSC C307331 -> (none); MPN (none) -> CL05B104KB54PNC
- D6: value Green -> LED; MPN (none) -> KT-0603R
- J1: MPN (none) -> M20-7910842R
- J2: MPN (none) -> M20-7911042R
- R2: LCSC C332662 -> (none); MPN (none) -> 0402WGF1001TCE
- R26: LCSC C25905 -> (none); MPN (none) -> RC0402FR-13100KL
- SW1: MPN (none) -> KSC741JLFS
- U1: MPN (none) -> STM32F042C6U6
- U11: LCSC C42379165 -> (none); MPN (none) -> TPSGM7227YUWQ10G
Connections:
- net GND: now also J2.10 (Pin_10), J2.3 (Pin_3); no longer J2.1 (Pin_1), J2.8 (Pin_8)
- net at J2.5 (Pin_5): now also JP2.1 (A); no longer JP3.1 (A)
- net at J2.6 (Pin_6): now also JP3.1 (A); no longer JP2.1 (A)
Other:
- note added: "1"
- note added: "2"
- note added: "3"
- note added: "4"
- note added: "5"
- note added: "6"
- note added: "7"
- note added: "8"
- note added: "9 10 11 12 13 14 15 16"
- company: (none) -> Rootkit Labs
- title: (none) -> Blackpants
- moved on the sheet: J1, J2, JP2, JP3
