File: hardware/keyboard.kicad_sch (KiCad schematic)
At the start: 10 parts, among them SW11 SW_Push, SW12 SW_Push, SW13 SW_Push, SW14 SW_Push, SW15 SW_Push, SW16 SW_Push, SW17 SW_Push, SW18 SW_Push, SW19 SW_Push

Commit message: R0.1 candidate
Parts:
- U14: now not fitted; now left out of the parts list
Other:
- note removed: "AI GEN CONTENT ^^"
- company: IUEngineering -> Rootkit Labs
- title: Keyboard -> Blackpants
