File: hardware/power.kicad_sch (KiCad schematic)
At the start: 48 parts, among them J8 USB_C_Receptacle_USB2.0_16P, Q1 AO3400A, U10 EL817S1C, U12 USBLC6-2SC6, U2 IP5306, U7 AOZ1280CI

Commit message: Passing DRC
Parts:
- removed C48: 100nF, Capacitor_SMD:C_0402_1005Metric, symbol Device:C_Small
- R16: footprint (none) -> Resistor_SMD:R_0402_1005Metric
Connections:
- net D+: now also U12.3 (I/O2); no longer U12.1 (I/O1)
- net D-: now also U12.1 (I/O1); no longer U12.3 (I/O2)
- net USB.D+: now also U12.4 (I/O2); no longer U12.6 (I/O1)
- net USB.D-: now also U12.6 (I/O1); no longer U12.4 (I/O2)
Other:
- moved on the sheet: BT1, C17, C18, C19, C2, C20, C21, C24, C25, C26, C45, C47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

Commit message: R0.1 candidate
Parts:
- BT1: Description_1 SMT Holder for 18650 Battery -> (none); JLCPCB_CORRECTION 0;0;-90 -> (none); LCSC C2988620 -> (none); MPN (none) -> BH-18650-B1BA002
- C1: MPN JMK105BJ105KV-F -> CL05B104KB54PNC
- C17, C2, C3: LCSC C96446 -> (none); MPN (none) -> CL10A106MA8NRNC
- C18, C19, C20, C21, C22, C24, C25, C26: LCSC C59461 -> (none); MPN (none) -> CL10A226MQ8NRNC
- C4, C5: MPN GRM188R61E106KA73J -> CL10A106MA8NRNC
- C45, C47, C49, C50: LCSC C307331 -> (none); MPN (none) -> CL05B104KB54PNC
- D2, D3, D4, D5: footprint Diode_SMD:D_0603_1608Metric -> LED_SMD:LED_0603_1608Metric; LCSC C2286 -> (none); MPN (none) -> KT-0603R
- D7: LCSC C2286 -> (none); MPN (none) -> KT-0603R
- F1: LCSC C20988 -> (none); MPN (none) -> SMD1206P200TF
- FB2: LCSC C76891 -> (none); MPN (none) -> BLM15PD121SN1D
- J8: LCSC C165948 -> (none); MPN (none) -> TYPE-C-31-M-12
- L1: LCSC C32712969 -> (none); MPN (none) -> RS0420-1R0MS
- PWR_BUTTON1: Availability Not in stock -> (none); Check_prices https://www.snapeda.com/parts/PTS847MM160LSMTR2%20LFS/C%252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 -> (none); Description_1 Tactile Switch SPST-NO Side Actuated Edge Mount, Right Angle -> (none); LCSC C2927781 -> (none); MANUFACTURER C&K -> (none); MAXIMUM_PACKAGE_HEIGHT 0.96 mm -> (none); MF C&K -> (none); MP PTS847MM160LSMTR2 LFS -> (none); MPN (none) -> PTS847MM160SMTR2LFS; PARTREV B -> (none); Package None -> (none); Price None -> (none); STANDARD Manufacturer Recommendations -> (none); SnapEDA_Link https://www.snapeda.com/parts/PTS847MM160LSMTR2%20LFS/C%252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 -> (none)
- Q1: JLCPCB_CORRECTION 0;0;180 -> (none); LCSC C20917 -> (none); MPN (none) -> AO3400A
- R11, R12: LCSC C25905 -> (none); MPN (none) -> RC0402FR-135K1L
- R14: LCSC C25157 -> (none); MPN (none) -> 0402WGJ020JTCE
- R15: LCSC C25744 -> (none); MPN (none) -> 0402WGF1002TCE
- R16: value 100k -> 100K; MPN (none) -> RC0402FR-13100KL
- R17: LCSC C332662 -> (none); MPN (none) -> RTT02R500FTH
- R38: LCSC C25082 -> (none); MPN (none) -> 0402WGF1500TCE
- R43: LCSC C11702 -> (none); MPN (none) -> 0402WGF1001TCE
- R50: LCSC C25117 -> (none); MPN (none) -> 0402WGF4700TCE
- U10: LCSC C2912100 -> (none); MPN (none) -> EL817S1(C)(TU)-F
- U12: LCSC C7519 -> (none); MPN (none) -> USBLC6-2SC6
- U2: JLCPCB_CORRECTION 0;0;-90 -> (none); MPN (none) -> IP5306
Other:
- company: (none) -> Rootkit Labs
- title: (none) -> Blackpants
