File: hardware/usb.kicad_sch (KiCad schematic)
At the start: 39 parts, among them J10 Conn_01x01_Pin, J4 USB_A, J5 USB_A, J6 Conn_01x01_Pin, J7 Conn_01x01_Pin, J9 Conn_01x01_Pin, U3 USB2514B_Bi, U4 MIC2026-1xM, U5 USBLC6-2SC6, U6 USBLC6-2SC6, U8 USBLC6-2SC6, Y1 24Mhz

Commit message: Passing DRC
Parts:
- added R24, R25: 100K, Resistor_SMD:R_0402_1005Metric, symbol Device:R_Small
- JP4, JP6: footprint (none) -> Jumper:SolderJumper-2_P1.3mm_Bridged_Pad1.0x1.5mm
Connections:
- net GND: now also R25.2
- net at J6.1 (Pin_1): now also R24.1
- new net USB_DET: R24.2, R25.1

Commit message: R0.1 candidate
Parts:
- added R27, R28: 100K, Resistor_SMD:R_0402_1005Metric, symbol Device:R_Small
- C12: LCSC C307331 -> (none); MPN (none) -> CL10A475MQ8NNNC
- C13, C14, C15, C16, C23, C27: LCSC C307331 -> (none); MPN (none) -> CL05B104KB54PNC
- C28, C29: LCSC C307331 -> (none); MPN (none) -> GRM1555C1H100FA01D
- C30: value 1.0uF -> 1uF; LCSC C307331 -> (none); MPN (none) -> CL05B104KB54PNC
- C31: value 0.1uF -> 100nF; LCSC C307331 -> (none); MPN (none) -> CL05B104KB54PNC
- D8: MPN (none) -> KT-0603R
- J4, J5: footprint Connector_USB:USB_A_Receptacle_GCT_USB1046 -> Connector_USB:USB_A_Receptacle_GCT_1; MPN (none) -> USB1046-GF-0190-L-B-A
- R10, R3, R4: LCSC C25905 -> (none); MPN (none) -> RC0402FR-135K1L
- R13, R20, R21, R24, R25, R6, R7, R9: LCSC C25905 -> (none); MPN (none) -> RC0402FR-13100KL
- R19: LCSC C25905 -> (none); MPN (none) -> 0402WGF1001TCE
- R5: LCSC C25905 -> (none); MPN (none) -> RC0402FR-131ML
- R8: LCSC C25905 -> (none); MPN (none) -> RC0402FR-1312KL
- U3: MPN (none) -> USB2514BI-AEZG-TR
- U4: MPN (none) -> MIC2026-1YM-TR
- U5, U6, U8: LCSC C7519 -> (none); MPN (none) -> USBLC6-2SC6
Connections:
- net +3V3: now also R27.1, R28.1
- net at U3.13 (OCS_N1), U4.2 (FLGA): now also R27.2
- net at U3.19 (OCS_N3), U4.3 (FLGB): now also R28.2
- net D-: now reaches J7.1 (Pin_1), U8.1 (I/O1)
- net D+: now reaches J9.1 (Pin_1), U8.3 (I/O2)
Other:
- note added: "1%"
- company: (none) -> Rootkit Labs
- title: (none) -> Blackpants
