File: ee/integrated/pmic.kicad_sch (KiCad schematic)
At the start: 52 parts, among them J501 Power Select, U501 LM66100DCK, U502 LM66100DCK, U503 TPS62095RGTR, U504 TPS62095RGTR, U505 AP131-25, U506 TPS62095RGTR, U507 TPS62095RGTR

Commit message: Added integrated parts.
Parts:
- removed J501: Power Select, Connector_PinHeader_2.54mm:PinHeader_1x03_P2.54mm_Vertical, symbol Connector:Conn_01x03_Pin
