File: ee/integrated/dsi_bridge.kicad_sch (KiCad schematic)
At the start: 15 parts, among them U15 AP3032

Commit message: Added a523 components.
Changed lines of the file:
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@@
 		(instances
 			(project "blackpants"
-				(path "/d0a98fce-b133-4503-8f8a-83b2a1eed591/d2fe0700-5ac0-49f8-be88-fb2ff272cc57"
+				(path "/d0a98fce-b133-4503-8f8a-83b2a1eed591/1d61bc11-ced6-4e86-9d3b-e9abe9ac6c2d/b9f74bdf-a26f-4f02-bb38-0b2e443d38e4"
 					(reference "D21")
 					(unit 1)
@@
 		(instances
 			(project "blackpants"
-				(path "/d0a98fce-b133-4503-8f8a-83b2a1eed591/d2fe0700-5ac0-49f8-be88-fb2ff272cc57"
+				(path "/d0a98fce-b133-4503-8f8a-83b2a1eed591/1d61bc11-ced6-4e86-9d3b-e9abe9ac6c2d/b9f74bdf-a26f-4f02-bb38-0b2e443d38e4"
 					(reference "#PWR072")
 					(unit 1)
@@
 		(instances
 			(project "blackpants"
-				(path "/d0a98fce-b133-4503-8f8a-83b2a1eed591/d2fe0700-5ac0-49f8-be88-fb2ff272cc57"
+				(path "/d0a98fce-b133-4503-8f8a-83b2a1eed591/1d61bc11-ced6-4e86-9d3b-e9abe9ac6c2d/b9f74bdf-a26f-4f02-bb38-0b2e443d38e4"
 					(reference "#PWR070")
 					(unit 1)
@@
 		(instances
 			(project "blackpants"
-				(path "/d0a98fce-b133-4503-8f8a-83b2a1eed591/d2fe0700-5ac0-49f8-be88-fb2ff272cc57"
+				(path "/d0a98fce-b133-4503-8f8a-83b2a1eed591/1d61bc11-ced6-4e86-9d3b-e9abe9ac6c2d/b9f74bdf-a26f-4f02-bb38-0b2e443d38e4"
 					(reference "U15")
 					(unit 1)
@@
 		(instances
 			(project "blackpants"
-				(path "/d0a98fce-b133-4503-8f8a-83b2a1eed591/d2fe0700-5ac0-49f8-be88-fb2ff272cc57"
+				(path "/d0a98fce-b133-4503-8f8a-83b2a1eed591/1d61bc11-ced6-4e86-9d3b-e9abe9ac6c2d/b9f74bdf-a26f-4f02-bb38-0b2e443d38e4"
 					(reference "#PWR074")
 					(unit 1)
@@
 		(instances
 			(project "blackpants"
-				(path "/d0a98fce-b133-4503-8f8a-83b2a1eed591/d2fe0700-5ac0-49f8-be88-fb2ff272cc57"
+				(path "/d0a98fce-b133-4503-8f8a-83b2a1eed591/1d61bc11-ced6-4e86-9d3b-e9abe9ac6c2d/b9f74bdf-a26f-4f02-bb38-0b2e443d38e4"
 					(reference "L3")
 					(unit 1)
@@
 		(instances
 			(project "blackpants"
-				(path "/d0a98fce-b133-4503-8f8a-83b2a1eed591/d2fe0700-5ac0-49f8-be88-fb2ff272cc57"
+				(path "/d0a98fce-b133-4503-8f8a-83b2a1eed591/1d61bc11-ced6-4e86-9d3b-e9abe9ac6c2d/b9f74bdf-a26f-4f02-bb38-0b2e443d38e4"
 					(reference "D17")
 					(unit 1)
@@
 		(instances
 			(project "blackpants"
-				(path "/d0a98fce-b133-4503-8f8a-83b2a1eed591/d2fe0700-5ac0-49f8-be88-fb2ff272cc57"
+				(path "/d0a98fce-b133-4503-8f8a-83b2a1eed591/1d61bc11-ced6-4e86-9d3b-e9abe9ac6c2d/b9f74bdf-a26f-4f02-bb38-0b2e443d38e4"
 					(reference "D16")
 					(unit 1)
@@
 		(instances
 			(project "blackpants"
-				(path "/d0a98fce-b133-4503-8f8a-83b2a1eed591/d2fe0700-5ac0-49f8-be88-fb2ff272cc57"
+				(path "/d0a98fce-b133-4503-8f8a-83b2a1eed591/1d61bc11-ced6-4e86-9d3b-e9abe9ac6c2d/b9f74bdf-a26f-4f02-bb38-0b2e443d38e4"
 					(reference "D15")
 					(unit 1)
@@
 		(instances
 			(project "blackpants"
-				(path "/d0a98fce-b133-4503-8f8a-83b2a1eed591/d2fe0700-5ac0-49f8-be88-fb2ff272cc57"
+				(path "/d0a98fce-b133-4503-8f8a-83b2a1eed591/1d61bc11-ced6-4e86-9d3b-e9abe9ac6c2d/b9f74bdf-a26f-4f02-bb38-0b2e443d38e4"
 					(reference "C32")
 					(unit 1)
@@
 		(instances
 			(project "blackpants"
-				(path "/d0a98fce-b133-4503-8f8a-83b2a1eed591/d2fe0700-5ac0-49f8-be88-fb2ff272cc57"
+				(path "/d0a98fce-b133-4503-8f8a-83b2a1eed591/1d61bc11-ced6-4e86-9d3b-e9abe9ac6c2d/b9f74bdf-a26f-4f02-bb38-0b2e443d38e4"
 					(reference "R22")
 					(unit 1)
@@
 		(instances
 			(project "blackpants"
-				(path "/d0a98fce-b133-4503-8f8a-83b2a1eed591/d2fe0700-5ac0-49f8-be88-fb2ff272cc57"
+				(path "/d0a98fce-b133-4503-8f8a-83b2a1eed591/1d61bc11-ced6-4e86-9d3b-e9abe9ac6c2d/b9f74bdf-a26f-4f02-bb38-0b2e443d38e4"
 					(reference "#PWR071")
 					(unit 1)
@@
 		(instances
 			(project "blackpants"
-				(path "/d0a98fce-b133-4503-8f8a-83b2a1eed591/d2fe0700-5ac0-49f8-be88-fb2ff272cc57"
+				(path "/d0a98fce-b133-4503-8f8a-83b2a1eed591/1d61bc11-ced6-4e86-9d3b-e9abe9ac6c2d/b9f74bdf-a26f-4f02-bb38-0b2e443d38e4"
 					(reference "#PWR0101")
 					(unit 1)
@@
 		(instances
 			(project "blackpants"
-				(path "/d0a98fce-b133-4503-8f8a-83b2a1eed591/d2fe0700-5ac0-49f8-be88-fb2ff272cc57"
+				(path "/d0a98fce-b133-4503-8f8a-83b2a1eed591/1d61bc11-ced6-4e86-9d3b-e9abe9ac6c2d/b9f74bdf-a26f-4f02-bb38-0b2e443d38e4"
 					(reference "D18")
 					(unit 1)
@@
 		(instances
 			(project "blackpants"
-				(path "/d0a98fce-b133-4503-8f8a-83b2a1eed591/d2fe0700-5ac0-49f8-be88-fb2ff272cc57"
+				(path "/d0a98fce-b133-4503-8f8a-83b2a1eed591/1d61bc11-ced6-4e86-9d3b-e9abe9ac6c2d/b9f74bdf-a26f-4f02-bb38-0b2e443d38e4"
 					(reference "C44")
 					(unit 1)
@@
 		(instances
 			(project "blackpants"
-				(path "/d0a98fce-b133-4503-8f8a-83b2a1eed591/d2fe0700-5ac0-49f8-be88-fb2ff272cc57"
+				(path "/d0a98fce-b133-4503-8f8a-83b2a1eed591/1d61bc11-ced6-4e86-9d3b-e9abe9ac6c2d/b9f74bdf-a26f-4f02-bb38-0b2e443d38e4"
 					(reference "D13")
 					(unit 1)
@@
 		(instances
 			(project "blackpants"
-				(path "/d0a98fce-b133-4503-8f8a-83b2a1eed591/d2fe0700-5ac0-49f8-be88-fb2ff272cc57"
+				(path "/d0a98fce-b133-4503-8f8a-83b2a1eed591/1d61bc11-ced6-4e86-9d3b-e9abe9ac6c2d/b9f74bdf-a26f-4f02-bb38-0b2e443d38e4"
 					(reference "R23")
 					(unit 1)
@@
 		(instances
 			(project "blackpants"
-				(path "/d0a98fce-b133-4503-8f8a-83b2a1eed591/d2fe0700-5ac0-49f8-be88-fb2ff272cc57"
+				(path "/d0a98fce-b133-4503-8f8a-83b2a1eed591/1d61bc11-ced6-4e86-9d3b-e9abe9ac6c2d/b9f74bdf-a26f-4f02-bb38-0b2e443d38e4"
 					(reference "D20")
 					(unit 1)
@@
 		(instances
 			(project "blackpants"
-				(path "/d0a98fce-b133-4503-8f8a-83b2a1eed591/d2fe0700-5ac0-49f8-be88-fb2ff272cc57"
+				(path "/d0a98fce-b133-4503-8f8a-83b2a1eed591/1d61bc11-ced6-4e86-9d3b-e9abe9ac6c2d/b9f74bdf-a26f-4f02-bb38-0b2e443d38e4"
 					(reference "#PWR068")
 					(unit 1)
@@
 		(instances
 			(project "blackpants"
-				(path "/d0a98fce-b133-4503-8f8a-83b2a1eed591/d2fe0700-5ac0-49f8-be88-fb2ff272cc57"
+				(path "/d0a98fce-b133-4503-8f8a-83b2a1eed591/1d61bc11-ced6-4e86-9d3b-e9abe9ac6c2d/b9f74bdf-a26f-4f02-bb38-0b2e443d38e4"
 					(reference "D19")
 					(unit 1)
@@
 		(instances
 			(project "blackpants"
-				(path "/d0a98fce-b133-4503-8f8a-83b2a1eed591/d2fe0700-5ac0-49f8-be88-fb2ff272cc57"
+				(path "/d0a98fce-b133-4503-8f8a-83b2a1eed591/1d61bc11-ced6-4e86-9d3b-e9abe9ac6c2d/b9f74bdf-a26f-4f02-bb38-0b2e443d38e4"
 					(reference "#PWR073")
 					(unit 1)
@@
 		(instances
 			(project "blackpants"
-				(path "/d0a98fce-b133-4503-8f8a-83b2a1eed591/d2fe0700-5ac0-49f8-be88-fb2ff272cc57"
+				(path "/d0a98fce-b133-4503-8f8a-83b2a1eed591/1d61bc11-ced6-4e86-9d3b-e9abe9ac6c2d/b9f74bdf-a26f-4f02-bb38-0b2e443d38e4"
 					(reference "#PWR069")
 					(unit 1)
@@
 		(instances
 			(project "blackpants"
-				(path "/d0a98fce-b133-4503-8f8a-83b2a1eed591/d2fe0700-5ac0-49f8-be88-fb2ff272cc57"
+				(path "/d0a98fce-b133-4503-8f8a-83b2a1eed591/1d61bc11-ced6-4e86-9d3b-e9abe9ac6c2d/b9f74bdf-a26f-4f02-bb38-0b2e443d38e4"
 					(reference "D22")
 					(unit 1)
 				)
+			)
+		)
+	)
+	(symbol
+		(lib_id "power:PWR_FLAG")
+		(at 81.28 59.69 0)
+		(unit 1)
+		(body_style 1)
+		(exclude_from_sim no)
+		(in_bom yes)
+		(on_board yes)
+		(in_pos_files yes)
+		(dnp no)
+		(property "Reference" "#FLG0906"
+			(at 81.28 49.53 0)
+			(hide yes)
+			(show_name no)
+			(do_not_autoplace no)
+			(effects
+				(font
+					(size 1.016 1.016)
+				)
+			)
+		)
+		(property "Value" "PWR_FLAG"
+			(at 81.28 52.07 0)
+			(hide yes)
+			(show_name no)
+			(do_not_autoplace no)
+			(effects
+				(font
+					(size 1.016 1.016)
+				)
+			)
+		)
+		(property "Footprint" ""
+			(at 81.28 52.07 0)
+			(hide yes)
+			(show_name no)
+			(do_not_autoplace no)
+			(effects
+				(font
+					(size 1.016 1.016)
+				)
+			)
+		)
+		(property "Datasheet" ""
+			(at 81.28 52.07 0)
+			(hide yes)
+			(show_name no)
+			(do_not_autoplace no)
+			(effects
+				(font
+					(size 1.016 1.016)
+				)
+			)
+		)
+		(property "Description" "Special symbol for telling ERC where power comes from"
+			(at 81.28 52.07 0)
+			(hide yes)
+			(show_name no)
+			(do_not_autoplace no)
+			(effects
+				(font
+					(size 1.016 1.016)
+				)
+			)
+		)
+		(property "ki_keywords" "flag power"
+			(at 81.28 52.07 0)
+			(hide yes)
+			(show_name no)
+			(do_not_autoplace no)
+			(effects
+				(font
+					(size 1.016 1.016)
+				)
+			)
+		)
+		(pin "1"
+		)
+		(instances
+			(project "blackpants"
+				(path "/d0a98fce-b133-4503-8f8a-83b2a1eed591/1d61bc11-ced6-4e86-9d3b-e9abe9ac6c2d/b9f74bdf-a26f-4f02-bb38-0b2e443d38e4"
+					(reference "#FLG0906")
+					(unit 1)
+				)
