File: ee/integrated/hardware.kicad_sch (KiCad schematic)
At the start: 14 parts, among them J101 USB_C_Receptacle_USB2.0_16P, J105 Micro_SD_Card_Det_Hirose_DM3AT

Commit message: Added a523 components.
Parts:
- removed C102: 100nF, Capacitor_SMD:C_0402_1005Metric, symbol Device:C_Small
- removed C103: 22uF, Capacitor_SMD:C_0402_1005Metric, symbol Device:C_Small
- removed J101: USB_C_Receptacle_USB2.0_16P, Connector_USB:USB_C_Receptacle_GCT_USB4105-xx-A_16P_TopMnt_Horizontal, symbol Connector:USB_C_Receptacle_USB2.0_16P
- removed J105: Micro_SD_Card_Det_Hirose_DM3AT, Connector_Card:microSD_HC_Hirose_DM3AT-SF-PEJM5, symbol Connector:Micro_SD_Card_Det_Hirose_DM3AT
- removed JP101, JP102: SolderJumper_2_Bridged, Jumper:SolderJumper-2_P1.3mm_Bridged_Pad1.0x1.5mm, symbol Jumper:SolderJumper_2_Bridged
- removed R101, R102: 5.6k, Resistor_SMD:R_0402_1005Metric, symbol Device:R_Small_US
- removed R103: 10k, Resistor_SMD:R_0402_1005Metric, symbol Device:R_Small_US
- removed R104, R105, R106, R107, R108: 100k, Resistor_SMD:R_0402_1005Metric, symbol Device:R_Small_US
Other:
- removed sheet A33_GPIO
- removed sheet A33_Power
- removed sheet A33_RAM
- removed sheet DDR3
- removed sheet DSI
- removed sheet PMIC
- removed sheet WiFi
- note removed: "3v3 @ 1A. 75uS startup time. 3v0 @ 1A. 75uS startup time. 2v5 @ 300mA. 75uS startup time. 1v35 @ 2A. 900uS startup time. 1v1 @ 4A. 900uS startup time."
- note removed: "Note, old resistors. SD_DAT[0..3] Pullup = 100k SD_CMD = Pullup 10k SD_DET = Pullup = 100k Make sure these are alright (with old sch), I want to swap them with a resisotor array."
- company: Interrupt Labs -> (none)
- title: Wifi Wart NFF -> A523 system
