File: ee/integrated/a523_always_on_io.kicad_sch (KiCad schematic)
At the start: 5 parts, among them U201 A523

Commit message: Working on the schematic.
Connections:
- net PMU_SCL renamed PMU.SCL
- net PMU_SDA renamed PMU.SDA
Changed lines of the file:
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@@
 		(at 114.3 88.9)
 	)
+	(bus_entry
+		(at 132.08 38.1)
+		(size -2.54 2.54)
+		(stroke
+			(width 0)
+			(type default)
+		)
+	)
+	(bus_entry
+		(at 132.08 35.56)
+		(size -2.54 2.54)
+		(stroke
+			(width 0)
+			(type default)
+		)
+	)
+	(bus_entry
+		(at 132.08 35.56)
+		(size -2.54 2.54)
+		(stroke
+			(width 0)
+			(type default)
+		)
+	)
+	(bus_entry
+		(at 132.08 38.1)
+		(size -2.54 2.54)
+		(stroke
+			(width 0)
+			(type default)
+		)
+	)
 	(wire
 		(pts
@@
 	(wire
 		(pts
-			(xy 114.3 40.64) (xy 119.38 40.64)
+			(xy 114.3 40.64) (xy 129.54 40.64)
 		)
 		(stroke
@@
 		)
 	)
+	(bus
+		(pts
+			(xy 132.08 38.1) (xy 132.08 33.02)
+		)
+		(stroke
+			(width 0)
+			(type default)
+		)
+	)
 	(wire
 		(pts
@@
 	(wire
 		(pts
-			(xy 114.3 38.1) (xy 119.38 38.1)
+			(xy 114.3 38.1) (xy 129.54 38.1)
 		)
 		(stroke
@@
 		)
 	)
-	(hierarchical_label "PMU_SCL"
-		(shape bidirectional)
+	(bus
+		(pts
+			(xy 132.08 33.02) (xy 134.62 33.02)
+		)
+		(stroke
+			(width 0)
+			(type default)
+		)
+	)
+	(label "PMU.SCL"
 		(at 119.38 38.1 0)
 		(effects
@@
 				(size 1.27 1.27)
 			)
-			(justify left)
-		)
-	)
-	(hierarchical_label "PMU_SDA"
-		(shape bidirectional)
+			(justify left bottom)
+		)
+	)
+	(label "PMU.SDA"
 		(at 119.38 40.64 0)
 		(effects
 			(font
+				(size 1.27 1.27)
+			)
+			(justify left bottom)
+		)
+	)
+	(hierarchical_label "PMU{I2C}"
+		(shape bidirectional)
+		(at 134.62 33.02 0)
+		(effects
+			(font
