File: ee/integrated/a523_axp323.kicad_sch (KiCad schematic)
At the start: 14 parts, among them U502 AXP323

Commit message: Working on the schematic.
Connections:
- net PMU_SCL renamed PMU.SCL
- net PMU_SDA renamed PMU.SDA
