File: ee/integrated/a523_axp323.kicad_sch (KiCad schematic)
At the start: 14 parts, among them U502 AXP323

Commit message: Worked on the layout.
Changed lines of the file:
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@@
 		)
 	)
+	(wire
+		(pts
+			(xy 139.7 82.55) (xy 139.7 86.36)
+		)
+		(stroke
+			(width 0)
+			(type default)
+		)
+	)
 	(bus
 		(pts
@@
 	(symbol
 		(lib_id "A523Power:VDD_DNR")
-		(at 139.7 86.36 0)
+		(at 139.7 82.55 0)
 		(unit 1)
 		(body_style 1)
@@
 		(dnp no)
 		(property "Reference" "#PWR0789626019"
-			(at 139.7 86.36 0)
+			(at 139.7 82.55 0)
 			(hide yes)
 			(show_name no)
@@
 		)
 		(property "Value" "VDD_DNR"
-			(at 139.7 82.55 0)
+			(at 139.7 78.74 0)
 			(show_name no)
 			(do_not_autoplace no)
@@
 		)
 		(property "Footprint" ""
-			(at 139.7 86.36 0)
+			(at 139.7 82.55 0)
 			(show_name no)
 			(do_not_autoplace no)
@@
 		)
 		(property "Datasheet" ""
-			(at 139.7 86.36 0)
+			(at 139.7 82.55 0)
 			(show_name no)
 			(do_not_autoplace no)
@@
 		)
 		(property "Description" ""
-			(at 139.7 86.36 0)
+			(at 139.7 82.55 0)
 			(show_name no)
 			(do_not_autoplace no)
