File: ee/integrated/a523_bucks.kicad_sch (KiCad schematic)
At the start: 11 parts, among them U501 AXP717C

Commit message: Working on the schematic.
Other:
- moved on the sheet: C511, C512, C513, C514, C515, C516, C517
