File: ee/integrated/a523_gpio.kicad_sch (KiCad schematic)
At the start: 3 parts, among them U201 A523

Commit message: Working on the schematic.
Connections:
- net A523_I2C1_SCL: no longer names the net of U201.J27 (PB4)
- net A523_I2C1_SDA: no longer names the net of U201.J28 (PB5)
- net SD0_CLK renamed SD0.CLK
- net SD0_CLK_SOC: no longer names the net of R203.1, U201.B12 (PF2)
- net SD0_CMD renamed SD0.CMD
- net SD0_D0 renamed SD0.D0
- net SD0_D1 renamed SD0.D1
- net SD0_D2 renamed SD0.D2
- net SD0_D3 renamed SD0.D3
- net SD0_DET renamed SD0.DET
Other:
- moved on the sheet: R203
