File: ee/integrated/a523_usb.kicad_sch (KiCad schematic)
At the start: 5 parts, among them U201 A523

Commit message: Working on the schematic.
Connections:
- net USB0_DM renamed USB0.DM
- net USB0_DP renamed USB0.DP
- net USB_HOST_DM renamed USB_HOST.DM
- net USB_HOST_DP renamed USB_HOST.DP
Other:
- moved on the sheet: U201H
