File: ee/integrated/console.kicad_sch (KiCad schematic)
At the start: 15 parts, among them J101 USB-C / recovery, J102 3.3V UART0: TX / RX / GND, J103 I2C1: 3V3 / SCL / SDA / GND, SW101 FEL / recovery, U101 USBLC6-2SC6, U402 CH340C

Commit message: Working on the schematic.
Parts:
- removed J102: 3.3V UART0: TX / RX / GND, Connector_PinHeader_2.54mm:PinHeader_1x03_P2.54mm_Vertical, symbol Connector_Generic:Conn_01x03
- removed J103: I2C1: 3V3 / SCL / SDA / GND, Connector_PinHeader_2.54mm:PinHeader_1x04_P2.54mm_Vertical, symbol Connector_Generic:Conn_01x04
- removed R125, R126: 4.7k, Resistor_SMD:R_0402_1005Metric, symbol Device:R_Small
Connections:
- net USB0_DM renamed USB0.DM
- net USB0_DP renamed USB0.DP
