File: ee/integrated/power.kicad_sch (KiCad schematic)
At the start: 49 parts, among them J8 USB_C_Receptacle_USB2.0_16P, U12 USBLC6-2SC6, U2 IP5306, U7 AOZ1280CI

Commit message: Added a523 components.
Parts:
- removed C1: 1uF, Capacitor_SMD:C_0402_1005Metric, symbol Device:C_Small
- removed C17, C2, C3: 10uF, Capacitor_SMD:C_0603_1608Metric, symbol Device:C
- removed C18, C19, C20, C21, C22, C24, C25, C26: 22uF, Capacitor_SMD:C_0603_1608Metric, symbol Device:C
- removed C4, C5: 10uF, Capacitor_SMD:C_0603_1608Metric, symbol Device:C_Small
- removed C45, C47, C49, C50: 100nF, Capacitor_SMD:C_0402_1005Metric, symbol Device:C_Small
- removed D1: MSS2P3, Diode_SMD:D_MicroSMP_AK, symbol Device:D_Schottky
- removed D2, D3, D4, D5: LED, LED_SMD:LED_0603_1608Metric, symbol Device:LED
- removed FB2: 120Ω@100MHz, Inductor_SMD:L_0402_1005Metric, symbol Device:FerriteBead_Small
- removed JP10, JP7, JP8, JP9: Jumper_2_Small_Open, Jumper:SolderJumper-2_P1.3mm_Open_RoundedPad1.0x1.5mm, symbol Jumper:Jumper_2_Small_Open
- removed L1: 1uH, Inductor_SMD:L_Changjiang_FXL0420, symbol Device:L
- removed L2: 2.2uH, Inductor_SMD:L_1008_2520Metric, symbol Device:L_Small
- removed R1: 49.9k, Resistor_SMD:R_0402_1005Metric, symbol Device:R_Small
- removed R11, R12: 5.1K, Resistor_SMD:R_0402_1005Metric, symbol Device:R_Small
- removed R14: 2, Resistor_SMD:R_0402_1005Metric, symbol Device:R
- removed R15: 10K, Resistor_SMD:R_0402_1005Metric, symbol Device:R_Small
- removed R16: 100K, Resistor_SMD:R_0402_1005Metric, symbol Device:R_Small
- removed R17: 0.5, Resistor_SMD:R_0402_1005Metric, symbol Device:R
- removed R18: 15.8k, Resistor_SMD:R_0402_1005Metric, symbol Device:R_Small
- removed R29, R30, R31, R32: 1K, Resistor_SMD:R_0402_1005Metric, symbol Device:R_Small
- removed U2: IP5306, Package_SO:HSOP-8-1EP_3.9x4.9mm_P1.27mm_EP2.41x3.1mm_ThermalVias, symbol IP5306:IP5306
- removed U7: AOZ1280CI, Package_TO_SOT_SMD:SOT-23-6, symbol Regulator_Switching:AOZ1280CI
- added C901: 100nF, Capacitor_SMD:C_0402_1005Metric, symbol Device:C_Small
- added C902: 10nF, Capacitor_SMD:C_0402_1005Metric, symbol Device:C_Small
- added D902: Charge status, LED_SMD:LED_0603_1608Metric, symbol Device:LED
- added R901, R902: 1k, Resistor_SMD:R_0402_1005Metric, symbol Device:R_Small
- added R903, R904: 470, Resistor_SMD:R_0402_1005Metric, symbol Device:R_Small
- added R905: 100k, Resistor_SMD:R_0402_1005Metric, symbol Device:R_Small
- added R906: 150k, Resistor_SMD:R_0402_1005Metric, symbol Device:R_Small
- added R907: 2.2k, Resistor_SMD:R_0402_1005Metric, symbol Device:R_Small
- added TH901: 10k @25C / cell-attached NTC, Connector_Wire:SolderWire-0.5sqmm_1x02_P4.6mm_D0.9mm_OD2.1mm, symbol Device:Thermistor_NTC
- BT1: value 18650 Cell -> Protected 18650 / 1S Li-ion; Description_1 (none) -> SMT Holder for 18650 Battery; MPN BH-18650-B1BA002 -> (none)
- F1: value Polyfuse -> 4A hold; footprint Fuse:Fuse_1206_3216Metric -> Fuse:Fuse_1812_4532Metric; MPN SMD1206P200TF -> (none)
- J8: value USB_C_Receptacle_USB2.0_16P -> USB-C / charge + keyboard; MPN TYPE-C-31-M-12 -> (none)
- PWR_BUTTON1: value PTS847MM160LSMTR2_LFS -> Power; footprint PTS847MM160LSMTR2_LFS:SW_PTS847MM160SMTR2_LFS -> PTS847MM160LSMTR2_LFS:SW_PTS847MM160LSMTR2_LFS; Availability (none) -> Not in stock; Check_prices (none) -> https://www.snapeda.com/parts/PTS847MM160LSMTR2%20LFS/C%252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; MANUFACTURER (none) -> C&K; MAXIMUM_PACKAGE_HEIGHT (none) -> 0.96 mm; MF (none) -> C&K; MP (none) -> PTS847MM160LSMTR2 LFS; MPN PTS847MM160SMTR2LFS -> (none); PARTREV (none) -> B; Package (none) -> None; Price (none) -> None; STANDARD (none) -> Manufacturer Recommendations; SnapEDA_Link (none) -> https://www.snapeda.com/parts/PTS847MM160LSMTR2%20LFS/C%252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
- U12: MPN USBLC6-2SC6 -> (none)
Connections:
- net UF is gone; now on net VBUS: J8.A4 (VBUS), J8.A9 (VBUS), J8.B4 (VBUS), J8.B9 (VBUS)
- net GND: now also J8.SH (SHIELD), PWR_BUTTON1.S1 (SHIELD), PWR_BUTTON1.S2 (SHIELD), C901.2, C902.2, R906.2, TH901.2; no longer J8.S1 (SHIELD)
- net VBUS: now also C901.1, R905.1
- net CC2: now reaches J8.B5 (CC2)
- net CC2: now also R902.1
- net CC1: now reaches J8.A5 (CC1)
- net CC1: now also R901.1
- net PWRON: now reaches PWR_BUTTON1.1, PWR_BUTTON1.3
- net +BATT renamed VBAT
- net D+ renamed SENSE_DP
- net SENSE_DP: now also R903.1
- net D- renamed SENSE_DM
- net SENSE_DM: now also R904.1
- net USB.D+ renamed MCU_USB_DP
- net USB.D- renamed MCU_USB_DM
- new net: D902.2 (A), R907.2
- new net BAT_TS: C902.1, TH901.1
- new net CHGLED_N: D902.1 (K)
- new net PMIC_CC1: R901.2
- new net PMIC_CC2: R902.2
- new net PMIC_USB_DM: R904.2
- new net PMIC_USB_DP: R903.2
- new net VBUS_PRESENT: R905.2, R906.1
- new net VSYS: R907.1
- no-connect marks 3 -> 2
Other:
- note added: "AXP717C is the only battery charger. The IP5306 path has been removed. J8 supplies VBUS only; peripheral +5V is a separate boost output. Set USB input/charge limits from the source capability and selected cell. TS: 50uA bias, 10k NTC; program temperature limits for the fitted curve."
- note removed: "USB C POWER"
- company: Rootkit Labs -> (none)
- title: Blackpants -> Battery, USB-C charging and keyboard USB

Commit message: Working on the schematic.
Other:
- moved on the sheet: R906
Changed lines of the file:
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@@
 	(wire
 		(pts
-			(xy 157.48 63.5) (xy 157.48 50.8)
+			(xy 157.48 53.34) (xy 157.48 50.8)
 		)
 		(stroke
@@
 		(pts
 			(xy 33.02 104.14) (xy 27.94 104.14)
+		)
+		(stroke
+			(width 0)
+			(type default)
+		)
+	)
+	(wire
+		(pts
+			(xy 157.48 58.42) (xy 157.48 59.69)
 		)
 		(stroke
@@
 				(size 1.27 1.27)
 			)
-			(justify left)
+			(justify left bottom)
 		)
 	)
@@
 				(size 1.27 1.27)
 			)
-			(justify left)
+			(justify left bottom)
 		)
 	)
@@
 				(size 1.27 1.27)
 			)
-			(justify left)
+			(justify left bottom)
 		)
 	)
@@
 		(dnp no)
 		(property "Reference" "D902"
-			(at 162.56 132.08 90)
+			(at 165.354 139.7 90)
 			(show_name no)
 			(do_not_autoplace no)
@@
 		(property "Value" "Charge status"
 			(at 162.56 134.62 90)
+			(hide yes)
 			(show_name no)
 			(do_not_autoplace no)
@@
 	(symbol
 		(lib_id "power:GND")
-		(at 157.48 68.58 0)
+		(at 157.48 59.69 0)
 		(unit 1)
 		(body_style 1)
@@
 		(dnp no)
 		(property "Reference" "#PWR772897923"
-			(at 157.48 68.58 0)
+			(at 157.48 59.69 0)
 			(hide yes)
 			(show_name no)
@@
 		)
 		(property "Value" "GND"
-			(at 157.48 72.39 0)
+			(at 157.48 63.5 0)
 			(hide yes)
 			(show_name no)
@@
 		)
 		(property "Footprint" ""
-			(at 157.48 68.58 0)
+			(at 157.48 59.69 0)
 			(show_name no)
 			(do_not_autoplace no)
@@
 		)
 		(property "Datasheet" ""
-			(at 157.48 68.58 0)
+			(at 157.48 59.69 0)
 			(show_name no)
 			(do_not_autoplace no)
@@
 		)
 		(property "Description" ""
-			(at 157.48 68.58 0)
+			(at 157.48 59.69 0)
 			(show_name no)
 			(do_not_autoplace no)
@@
 	(symbol
 		(lib_id "Device:R_Small")
-		(at 157.48 66.04 0)
+		(at 157.48 55.88 0)
 		(unit 1)
 		(body_style 1)
@@
 		(dnp no)
 		(property "Reference" "R906"
-			(at 161.29 64.77 0)
+			(at 161.29 54.61 0)
 			(show_name no)
 			(do_not_autoplace no)
@@
 		)
 		(property "Value" "150k"
-			(at 161.29 67.31 0)
+			(at 161.29 57.15 0)
 			(show_name no)
 			(do_not_autoplace no)
@@
 		)
 		(property "Footprint" "Resistor_SMD:R_0402_1005Metric"
-			(at 161.29 67.31 0)
+			(at 161.29 57.15 0)
 			(hide yes)
 			(show_name no)
@@
 		)
 		(property "Datasheet" ""
-			(at 161.29 67.31 0)
+			(at 161.29 57.15 0)
 			(hide yes)
 			(show_name no)
@@
 		)
 		(property "Description" "Resistor, small symbol"
-			(at 161.29 67.31 0)
+			(at 161.29 57.15 0)
 			(hide yes)
 			(show_name no)
@@
 		)
 		(property "ki_keywords" "R resistor"
-			(at 161.29 67.31 0)
+			(at 161.29 57.15 0)
 			(hide yes)
 			(show_name no)
@@
 		)
 		(property "ki_fp_filters" "R_*"
-			(at 161.29 67.31 0)
-			(hide yes)
-			(show_name no)
+			(at 161.29 57.15 0)
+			(hide yes)
+			(show_name no)
