File: ee/integrated/sdcard.kicad_sch (KiCad schematic)
At the start: 9 parts, among them J105 microSD / boot

Commit message: Working on the schematic.
Connections:
- net SD0_CLK renamed SD0.CLK
- net SD0_CMD renamed SD0.CMD
- net SD0_D0 renamed SD0.D0
- net SD0_D1 renamed SD0.D1
- net SD0_D2 renamed SD0.D2
- net SD0_D3 renamed SD0.D3
- net SD0_DET renamed SD0.DET
Other:
- note removed: "PF0..PF5 SDC0, 3.3V removable card. PF6 detect is active low. Clock series resistor R203 is at the SoC. No clock pull-up. C102/C103 at the socket. Configure card-detect pull-up before use."
