File: ee/integrated/a523_charger.kicad_sch (KiCad schematic)
At the start: 16 parts, among them U501 AXP717C

Commit message: Working on the schematic.
Connections:
- net PMU_SCL: no longer U501.52 (SCK)
- net PMU_SDA: no longer U501.51 (SDA)
- new net PMU.SCL: U501.52 (SCK)
- new net PMU.SDA: U501.51 (SDA)

Commit message: Cleaned up routing.
Connections:
- net PMU_SCL is gone; now on net PMU.SCL: R501.2
- net PMU_SDA is gone; now on net PMU.SDA: R502.2
Changed lines of the file:
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@@
+		)
+	)
+	(label "PMU.SDA"
+		(at 86.36 143.51 0)
+		(effects
+			(font
+				(size 1.27 1.27)
+			)
+			(justify left bottom)
+		)
+	)
+	(label "PMU.SCL"
+		(at 43.18 143.51 0)
+		(effects
+			(font
+				(size 1.27 1.27)
+			)
+			(justify left bottom)
 		)
 	)
@@
 		(effects
 			(font
-				(size 1.27 1.27)
-			)
-			(justify left)
-		)
-	)
-	(hierarchical_label "PMU_SDA"
-		(shape bidirectional)
-		(at 86.36 143.51 0)
-		(effects
-			(font
-				(size 1.27 1.27)
-			)
-			(justify left)
-		)
-	)
-	(hierarchical_label "PMU_SCL"
-		(shape bidirectional)
-		(at 43.18 143.51 0)
-		(effects
-			(font
