File: ee/integrated/stm32.kicad_sch (KiCad schematic)
At the start: 17 parts, among them J3 Conn_ARM_SWD_TagConnect_TC203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, SW1 SW_Push, U1 STM32F042C6Ux, U11 TPSGM7227YUWQ10G

Commit message: Cleaned up routing.
Connections:
- net LED: now reaches R2.1, U1.40 (PB4)
Other:
- moved on the sheet: D6, R2
Changed lines of the file:
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@@
 	)
 	(bus_entry
+		(at 123.19 129.54)
+		(size -2.54 -2.54)
+		(stroke
+			(width 0)
+			(type default)
+		)
+	)
+	(bus_entry
 		(at 59.944 44.958)
 		(size 2.54 2.54)
@@
 	)
 	(bus_entry
+		(at 123.19 127)
+		(size -2.54 -2.54)
+		(stroke
+			(width 0)
+			(type default)
+		)
+	)
+	(bus_entry
 		(at 59.944 83.058)
 		(size 2.54 2.54)
@@
 	(wire
 		(pts
-			(xy 113.03 147.32) (xy 113.03 144.78)
+			(xy 113.03 170.18) (xy 113.03 167.64)
 		)
 		(stroke
@@
 	(wire
 		(pts
-			(xy 113.03 111.76) (xy 113.03 124.46)
+			(xy 113.03 144.78) (xy 113.03 147.32)
 		)
 		(stroke
@@
 	(wire
 		(pts
+			(xy 123.19 127) (xy 134.62 127)
+		)
+		(stroke
+			(width 0)
+			(type default)
+		)
+	)
+	(wire
+		(pts
 			(xy 121.92 67.31) (xy 121.92 71.12)
 		)
@@
 	(wire
 		(pts
-			(xy 134.62 111.76) (xy 113.03 111.76)
-		)
-		(stroke
-			(width 0)
-			(type default)
-		)
-	)
-	(wire
-		(pts
 			(xy 33.02 114.3) (xy 33.02 116.84)
 		)
@@
 	(wire
 		(pts
-			(xy 134.62 127) (xy 130.81 127)
-		)
-		(stroke
-			(width 0)
-			(type default)
-		)
-	)
-	(wire
-		(pts
 			(xy 144.78 64.77) (xy 147.32 64.77)
 		)
@@
 	(wire
 		(pts
+			(xy 130.81 111.76) (xy 134.62 111.76)
+		)
+		(stroke
+			(width 0)
+			(type default)
+		)
+	)
+	(wire
+		(pts
 			(xy 187.96 114.3) (xy 189.23 114.3)
 		)
@@
 		)
 	)
+	(bus
+		(pts
+			(xy 120.65 119.38) (xy 120.65 124.46)
+		)
+		(stroke
+			(width 0)
+			(type default)
+		)
+	)
 	(wire
 		(pts
@@
 		)
 	)
+	(bus
+		(pts
+			(xy 116.84 119.38) (xy 120.65 119.38)
+		)
+		(stroke
+			(width 0)
+			(type default)
+		)
+	)
 	(wire
 		(pts
@@
 	(wire
 		(pts
-			(xy 113.03 132.08) (xy 113.03 137.16)
+			(xy 113.03 154.94) (xy 113.03 160.02)
 		)
 		(stroke
@@
 	(wire
 		(pts
-			(xy 134.62 129.54) (xy 130.81 129.54)
-		)
-		(stroke
-			(width 0)
-			(type default)
-		)
-	)
-	(wire
-		(pts
 			(xy 134.62 106.68) (xy 130.81 106.68)
 		)
@@
 	(wire
 		(pts
+			(xy 123.19 129.54) (xy 134.62 129.54)
+		)
+		(stroke
+			(width 0)
+			(type default)
+		)
+	)
+	(wire
+		(pts
 			(xy 134.62 121.92) (xy 130.81 121.92)
 		)
@@
 		)
 	)
+	(bus
+		(pts
+			(xy 120.65 124.46) (xy 120.65 127)
+		)
+		(stroke
+			(width 0)
+			(type default)
+		)
+	)
 	(wire
 		(pts
@@
 		)
 	)
+	(label "LED"
+		(at 113.03 144.78 180)
+		(effects
+			(font
+				(size 1.27 1.27)
+			)
+			(justify right bottom)
+		)
+	)
 	(label "USB_DET"
 		(at 130.81 91.44 180)
@@
 		)
 	)
+	(label "LED"
+		(at 130.81 111.76 180)
+		(effects
+			(font
+				(size 1.27 1.27)
+			)
+			(justify right bottom)
+		)
+	)
 	(label "COL_1"
 		(at 130.81 104.14 180)
@@
 		)
 	)
+	(hierarchical_label "I2C{SCL SDA}"
+		(shape bidirectional)
+		(at 116.84 119.38 180)
+		(effects
+			(font
+				(size 1.27 1.27)
+			)
+			(justify right)
+		)
+	)
 	(hierarchical_label "USB3.D-"
 		(shape bidirectional)
@@
 	(symbol
 		(lib_id "power:GND")
-		(at 113.03 147.32 0)
+		(at 113.03 170.18 0)
 		(unit 1)
 		(body_style 1)
@@
 		(fields_autoplaced yes)
 		(property "Reference" "#PWR018"
-			(at 113.03 153.67 0)
+			(at 113.03 176.53 0)
 			(hide yes)
 			(show_name no)
@@
 		)
 		(property "Value" "GND"
-			(at 113.03 152.4 0)
+			(at 113.03 175.26 0)
 			(hide yes)
 			(show_name no)
@@
 		)
 		(property "Footprint" ""
-			(at 113.03 147.32 0)
+			(at 113.03 170.18 0)
 			(hide yes)
 			(show_name no)
@@
 		)
 		(property "Datasheet" ""
-			(at 113.03 147.32 0)
+			(at 113.03 170.18 0)
 			(hide yes)
 			(show_name no)
@@
 		)
 		(property "Description" "Power symbol creates a global label with name \"GND\" , ground"
-			(at 113.03 147.32 0)
+			(at 113.03 170.18 0)
 			(hide yes)
 			(show_name no)
@@
 	(symbol
 		(lib_id "Device:R")
-		(at 113.03 128.27 0)
+		(at 113.03 151.13 0)
 		(unit 1)
 		(body_style 1)
@@
 		(fields_autoplaced yes)
 		(property "Reference" "R2"
-			(at 115.57 126.9999 0)
+			(at 115.57 149.8599 0)
 			(show_name no)
 			(do_not_autoplace no)
@@
 		)
 		(property "Value" "1k"
-			(at 115.57 129.5399 0)
+			(at 115.57 152.3999 0)
 			(show_name no)
 			(do_not_autoplace no)
@@
 		)
 		(property "Footprint" "Resistor_SMD:R_0402_1005Metric"
-			(at 111.252 128.27 90)
+			(at 111.252 151.13 90)
 			(hide yes)
 			(show_name no)
@@
 		)
 		(property "Datasheet" ""
-			(at 113.03 128.27 0)
+			(at 113.03 151.13 0)
 			(hide yes)
 			(show_name no)
@@
 		)
 		(property "Description" "Resistor"
-			(at 113.03 128.27 0)
+			(at 113.03 151.13 0)
 			(hide yes)
 			(show_name no)
@@
 		)
 		(property "LCSC" ""
-			(at 113.03 128.27 0)
+			(at 113.03 151.13 0)
 			(hide yes)
 			(show_name no)
@@
 		)
 		(property "MPN" "0402WGF1001TCE"
-			(at 113.03 128.27 0)
+			(at 113.03 151.13 0)
 			(hide yes)
 			(show_name no)
@@
 	(symbol
 		(lib_id "Device:LED")
-		(at 113.03 140.97 90)
+		(at 113.03 163.83 90)
 		(unit 1)
 		(body_style 1)
@@
 		(fields_autoplaced yes)
 		(property "Reference" "D6"
-			(at 116.84 141.2874 90)
+			(at 116.84 164.1474 90)
 			(show_name no)
 			(do_not_autoplace no)
@@
 		)
 		(property "Value" "LED"
-			(at 116.84 143.8274 90)
+			(at 116.84 166.6874 90)
 			(show_name no)
 			(do_not_autoplace no)
@@
 		)
 		(property "Footprint" "LED_SMD:LED_0603_1608Metric"
-			(at 113.03 140.97 0)
+			(at 113.03 163.83 0)
 			(hide yes)
 			(show_name no)
@@
 		)
 		(property "Datasheet" ""
-			(at 113.03 140.97 0)
+			(at 113.03 163.83 0)
 			(hide yes)
 			(show_name no)
@@
 		)
 		(property "Description" "Light emitting diode"
-			(at 113.03 140.97 0)
+			(at 113.03 163.83 0)
 			(hide yes)
 			(show_name no)
@@
 		)
 		(property "MPN" "KT-0603R"
-			(at 113.03 140.97 90)
+			(at 113.03 163.83 90)
 			(hide yes)
 			(show_name no)
