File: ee/integrated/usb.kicad_sch (KiCad schematic)
At the start: 36 parts, among them J4 USB_A, J5 USB_A, U3 USB2514B_Bi, U4 MIC2026-1xM, U5 USBLC6-2SC6, U6 USBLC6-2SC6, Y1 24Mhz

Commit message: Added a523 components.
Parts:
- removed R20, R21: 100K, Resistor_SMD:R_0402_1005Metric, symbol Device:R_Small
- J4, J5: footprint Connector_USB:USB_A_Receptacle_GCT_1 -> blackpants:USB_A_Receptacle_GCT_1
Connections:
- net HUB_CONSOLE_DM: now reaches U3.8 (USBDM_DN4/PRT_DIS_M4)
- net HUB_CONSOLE_DP: now reaches U3.9 (USBDP_DN4/PRT_DIS_P4)
- net USB3.D+ renamed HUB_MCU_DP
- net USB3.D- renamed HUB_MCU_DM
- net USBUP.D+ renamed USB_HOST_DP
- net USBUP.D- renamed USB_HOST_DM
- no-connect marks 0 -> 2

Commit message: Working on the schematic.
Connections:
- net USB_HOST_DM renamed USB_HOST.DM
- net USB_HOST_DP renamed USB_HOST.DP
Changed lines of the file:
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@@
+	)
+	(bus_entry
+		(at 55.88 105.41)
+		(size 2.54 2.54)
+		(stroke
+			(width 0)
+			(type default)
+		)
+	)
+	(bus_entry
+		(at 55.88 107.95)
+		(size 2.54 2.54)
+		(stroke
+			(width 0)
+			(type default)
+		)
 	)
 	(bus_entry
@@
 	(wire
 		(pts
-			(xy 72.39 110.49) (xy 87.63 110.49)
-		)
-		(stroke
-			(width 0)
-			(type default)
-		)
-	)
-	(wire
-		(pts
 			(xy 15.24 162.56) (xy 15.24 168.91)
 		)
@@
 		)
 	)
+	(bus
+		(pts
+			(xy 55.88 104.14) (xy 55.88 107.95)
+		)
+		(stroke
+			(width 0)
+			(type default)
+		)
+	)
 	(wire
 		(pts
@@
 	(wire
 		(pts
-			(xy 72.39 107.95) (xy 87.63 107.95)
-		)
-		(stroke
-			(width 0)
-			(type default)
-		)
-	)
-	(wire
-		(pts
 			(xy 43.18 144.78) (xy 50.8 144.78)
 		)
@@
 	(wire
 		(pts
+			(xy 58.42 107.95) (xy 87.63 107.95)
+		)
+		(stroke
+			(width 0)
+			(type default)
+		)
+	)
+	(wire
+		(pts
 			(xy 85.09 123.19) (xy 87.63 123.19)
 		)
@@
 	(wire
 		(pts
+			(xy 58.42 110.49) (xy 87.63 110.49)
+		)
+		(stroke
+			(width 0)
+			(type default)
+		)
+	)
+	(wire
+		(pts
 			(xy 86.36 55.88) (xy 86.36 58.42)
 		)
@@
 		(pts
 			(xy 234.95 82.55) (xy 254 82.55)
+		)
+		(stroke
+			(width 0)
+			(type default)
+		)
+	)
+	(bus
+		(pts
+			(xy 54.61 104.14) (xy 55.88 104.14)
 		)
 		(stroke
@@
 	(label "~{RESET}"
 		(at 78.74 115.57 0)
+		(effects
+			(font
+				(size 1.27 1.27)
+			)
+			(justify left bottom)
+		)
+	)
+	(label "USB_HOST.DM"
+		(at 59.69 107.95 0)
+		(effects
+			(font
+				(size 1.27 1.27)
+			)
+			(justify left bottom)
+		)
+	)
+	(label "USB_HOST.DP"
+		(at 59.69 110.49 0)
 		(effects
 			(font
@@
 		)
 	)
-	(hierarchical_label "USB_HOST_DP"
+	(hierarchical_label "USB_HOST{USB}"
 		(shape bidirectional)
-		(at 72.39 110.49 180)
+		(at 54.61 104.14 180)
 		(effects
 			(font
-				(size 1.27 1.27)
-			)
-			(justify right)
-		)
-	)
-	(hierarchical_label "USB_HOST_DM"
-		(shape bidirectional)
-		(at 72.39 107.95 180)
-		(effects
-			(font

Commit message: Removed USB sheets and moved the parts to the main sheets.
Connections:
- net HUB_CONSOLE_DM: no longer names the net of U3.8 (USBDM_DN4/PRT_DIS_M4)
- net HUB_CONSOLE_DP: no longer names the net of U3.9 (USBDP_DN4/PRT_DIS_P4)
Changed lines of the file:
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@@
-		)
-	)
-	(hierarchical_label "HUB_CONSOLE_DP"
-		(shape bidirectional)
-		(at 157.48 143.51 0)
-		(effects
-			(font
-				(size 1.27 1.27)
-			)
-			(justify left)
 		)
 	)
@@
 		(effects
 			(font
-				(size 1.27 1.27)
-			)
-			(justify left)
-		)
-	)
-	(hierarchical_label "HUB_CONSOLE_DM"
-		(shape bidirectional)
-		(at 157.48 140.97 0)
-		(effects
-			(font

Commit message: Cleaned up routing.
Connections:
- net +3V3: now also U3.8 (USBDM_DN4/PRT_DIS_M4), U3.9 (USBDP_DN4/PRT_DIS_P4)
Changed lines of the file:
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@@
+	)
+	(junction
+		(at 146.05 140.97)
+		(diameter 0)
+		(color 0 0 0 0)
 	)
 	(junction
@@
 	(wire
 		(pts
+			(xy 143.51 143.51) (xy 146.05 143.51)
+		)
+		(stroke
+			(width 0)
+			(type default)
+		)
+	)
+	(wire
+		(pts
 			(xy 87.63 153.67) (xy 86.36 153.67)
 		)
@@
 	(wire
 		(pts
+			(xy 146.05 140.97) (xy 148.59 140.97)
+		)
+		(stroke
+			(width 0)
+			(type default)
+		)
+	)
+	(wire
+		(pts
 			(xy 76.2 87.63) (xy 76.2 88.9)
 		)
@@
 	(wire
 		(pts
-			(xy 143.51 143.51) (xy 157.48 143.51)
-		)
-		(stroke
-			(width 0)
-			(type default)
-		)
-	)
-	(wire
-		(pts
 			(xy 43.18 144.78) (xy 43.18 147.32)
 		)
@@
 	(wire
 		(pts
+			(xy 148.59 139.7) (xy 148.59 140.97)
+		)
+		(stroke
+			(width 0)
+			(type default)
+		)
+	)
+	(wire
+		(pts
 			(xy 71.12 63.5) (xy 71.12 66.04)
 		)
@@
 	(wire
 		(pts
+			(xy 146.05 143.51) (xy 146.05 140.97)
+		)
+		(stroke
+			(width 0)
+			(type default)
+		)
+	)
+	(wire
+		(pts
 			(xy 58.42 144.78) (xy 58.42 147.32)
 		)
@@
 	(wire
 		(pts
-			(xy 143.51 140.97) (xy 157.48 140.97)
+			(xy 143.51 140.97) (xy 146.05 140.97)
 		)
 		(stroke
@@
 					(unit 1)
 				)
+			)
+		)
+	)
+	(symbol
+		(lib_id "power:+5V")
+		(at 148.59 139.7 0)
+		(unit 1)
+		(body_style 1)
+		(exclude_from_sim no)
+		(in_bom yes)
+		(on_board yes)
+		(in_pos_files yes)
+		(dnp no)
+		(property "Reference" "#PWR047"
+			(at 148.59 143.51 0)
+			(hide yes)
+			(show_name no)
+			(do_not_autoplace no)
+			(effects
+				(font
+					(size 1.27 1.27)
+				)
+			)
+		)
+		(property "Value" "+3V3"
+			(at 152.146 137.668 0)
+			(show_name no)
+			(do_not_autoplace no)
+			(effects
+				(font
+					(size 1.27 1.27)
+				)
+			)
+		)
+		(property "Footprint" ""
+			(at 148.59 139.7 0)
+			(hide yes)
+			(show_name no)
+			(do_not_autoplace no)
+			(effects
+				(font
+					(size 1.27 1.27)
+				)
+			)
+		)
+		(property "Datasheet" ""
+			(at 148.59 139.7 0)
+			(hide yes)
+			(show_name no)
+			(do_not_autoplace no)
+			(effects
+				(font
+					(size 1.27 1.27)
+				)
+			)
+		)
+		(property "Description" ""
+			(at 148.59 139.7 0)
+			(show_name no)
+			(do_not_autoplace no)
+			(effects
+				(font
+					(size 1.27 1.27)
+				)
+			)
+		)
+		(pin "1"
+		)
+		(instances
+			(project "blackpants"
+				(path "/d0a98fce-b133-4503-8f8a-83b2a1eed591/773f8af3-a641-4fcc-9414-9cf290a67b77"
+					(reference "#PWR047")
+					(unit 1)
+				)
