File: ee/integrated/a523_analog.kicad_sch (KiCad schematic)
At the start: 17 parts, among them U201 A523

Commit message: Worked on the layout.
Parts:
- removed C282: 10uF, Capacitor_SMD:C_0402_1005Metric, symbol Device:C_Small
