File: ee/integrated/a523_ldos.kicad_sch (KiCad schematic)
At the start: 17 parts, among them U501 AXP717C

Commit message: Worked on the layout.
Parts:
- removed C523, C524, C527, C529, C530, C532, C534: 2.2uF, Capacitor_SMD:C_0402_1005Metric, symbol Device:C_Small
Connections:
- net ALDO1_UNUSED: no longer names the net of U501.13 (ALDO1)
- net BLDO3_UNUSED: no longer names the net of U501.21 (BLDO3)
- net BLDO4_UNUSED: no longer names the net of U501.22 (BLDO4)
- net CLDO2_UNUSED: no longer names the net of U501.24 (CLDO2)
- net VCC_LCD: no longer names the net of U501.27 (CLDO4)
- net VCC_PE: no longer names the net of U501.14 (ALDO2)
- net VCC_PG: no longer names the net of U501.18 (BLDO1)
- no-connect marks 0 -> 7
Other:
- moved on the sheet: C520, C521, C522
