File: ee/integrated/a523_wifi_io.kicad_sch (KiCad schematic)
At the start: 7 parts, among them U201 A523

Commit message: Working on the schematic.
Connections:
- net BT_CTS_N renamed BT.~{CTS}
- net BT_RTS_N renamed BT.~{RTS}
- net BT_RXD renamed BT.RX
- net BT_TXD renamed BT.TX
- net SD1_CLK: no longer names the net of R208.2
- net SD1_CLK: now also U201.R1 (PG0)
- net SD1_CLK_SOC renamed SD1.CLK
- net SD1.CLK: no longer U201.R1 (PG0)
- net SD1_CMD renamed SD1.CMD
- net SD1_D0 renamed SD1.D0
- net SD1_D1 renamed SD1.D1
- net SD1_D2 renamed SD1.D2
- net SD1_D3 renamed SD1.D3
Other:
- moved on the sheet: R208

Commit message: Worked on the layout.
Connections:
- net VCC_PG renamed +3V3
Other:
- moved on the sheet: C266
Changed lines of the file:
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@@
+		)
+	)
+	(wire
+		(pts
+			(xy 48.26 72.39) (xy 48.26 76.2)
+		)
+		(stroke
+			(width 0)
+			(type default)
 		)
 	)
@@
 	(wire
 		(pts
-			(xy 182.88 43.18) (xy 182.88 44.45)
+			(xy 33.02 87.63) (xy 33.02 88.9)
 		)
 		(stroke
@@
 	(wire
 		(pts
-			(xy 182.88 38.1) (xy 182.88 35.56)
+			(xy 33.02 82.55) (xy 33.02 80.01)
 		)
 		(stroke
@@
 	)
 	(symbol
-		(lib_id "A523Power:VCC_PG")
-		(at 48.26 76.2 90)
-		(unit 1)
-		(body_style 1)
-		(exclude_from_sim no)
-		(in_bom no)
-		(on_board yes)
-		(in_pos_files yes)
-		(dnp no)
-		(property "Reference" "#PWR0108701807"
-			(at 48.26 76.2 0)
-			(hide yes)
-			(show_name no)
-			(do_not_autoplace no)
-			(effects
-				(font
-					(size 1.016 1.016)
-				)
-			)
-		)
-		(property "Value" "VCC_PG"
-			(at 41.415 76.2 90)
-			(show_name no)
-			(do_not_autoplace no)
-			(effects
-				(font
-					(size 1.016 1.016)
-				)
-			)
-		)
-		(property "Footprint" ""
-			(at 48.26 76.2 0)
-			(show_name no)
-			(do_not_autoplace no)
-			(effects
-				(font
-					(size 1.27 1.27)
-				)
-			)
-		)
-		(property "Datasheet" ""
-			(at 48.26 76.2 0)
-			(show_name no)
-			(do_not_autoplace no)
-			(effects
-				(font
-					(size 1.27 1.27)
-				)
-			)
-		)
-		(property "Description" ""
-			(at 48.26 76.2 0)
-			(show_name no)
-			(do_not_autoplace no)
-			(effects
-				(font
-					(size 1.27 1.27)
-				)
-			)
-		)
-		(pin "1"
-		)
-		(instances
-			(project "blackpants"
-				(path "/d0a98fce-b133-4503-8f8a-83b2a1eed591/7b29c749-8ab5-43b5-aee9-52b112811e58"
-					(reference "#PWR0108701807")
-					(unit 1)
-				)
-			)
-		)
-	)
-	(symbol
 		(lib_id "Device:C_Small")
-		(at 182.88 40.64 0)
+		(at 33.02 85.09 0)
+		(mirror y)
 		(unit 1)
 		(body_style 1)
@@
 		(dnp no)
 		(property "Reference" "C266"
-			(at 186.69 39.37 0)
+			(at 29.21 83.82 0)
 			(show_name no)
 			(do_not_autoplace no)
@@
 		)
 		(property "Value" "100nF"
-			(at 186.69 41.91 0)
+			(at 29.21 86.36 0)
 			(show_name no)
 			(do_not_autoplace no)
@@
 		)
 		(property "Footprint" "Capacitor_SMD:C_0201_0603Metric"
-			(at 186.69 41.91 0)
+			(at 29.21 86.36 0)
 			(hide yes)
 			(show_name no)
@@
 		)
 		(property "Datasheet" ""
-			(at 186.69 41.91 0)
+			(at 29.21 86.36 0)
 			(hide yes)
 			(show_name no)
@@
 		)
 		(property "Description" "Unpolarized capacitor, small symbol"
-			(at 186.69 41.91 0)
+			(at 29.21 86.36 0)
 			(hide yes)
 			(show_name no)
@@
 		)
 		(property "ki_keywords" "capacitor cap"
-			(at 186.69 41.91 0)
+			(at 29.21 86.36 0)
 			(hide yes)
 			(show_name no)
@@
 		)
 		(property "ki_fp_filters" "C_*"
-			(at 186.69 41.91 0)
+			(at 29.21 86.36 0)
 			(hide yes)
 			(show_name no)
@@
 		)
 		(property "Voltage" "10V"
-			(at 186.69 41.91 0)
+			(at 29.21 86.36 0)
 			(hide yes)
 			(show_name no)
@@
 		)
 		(property "Dielectric" "X5R/X7R"
-			(at 186.69 41.91 0)
+			(at 29.21 86.36 0)
 			(hide yes)
 			(show_name no)
@@
 	(symbol
 		(lib_id "power:GND")
-		(at 182.88 44.45 0)
+		(at 33.02 88.9 0)
+		(mirror y)
 		(unit 1)
 		(body_style 1)
@@
 		(dnp no)
 		(property "Reference" "#PWR0869997685"
-			(at 182.88 44.45 0)
+			(at 33.02 88.9 0)
 			(hide yes)
 			(show_name no)
@@
 		)
 		(property "Value" "GND"
-			(at 182.88 48.26 0)
+			(at 33.02 92.71 0)
 			(hide yes)
 			(show_name no)
@@
 		)
 		(property "Footprint" ""
-			(at 182.88 44.45 0)
+			(at 33.02 88.9 0)
 			(show_name no)
 			(do_not_autoplace no)
@@
 		)
 		(property "Datasheet" ""
-			(at 182.88 44.45 0)
+			(at 33.02 88.9 0)
 			(show_name no)
 			(do_not_autoplace no)
@@
 		)
 		(property "Description" ""
-			(at 182.88 44.45 0)
+			(at 33.02 88.9 0)
 			(show_name no)
 			(do_not_autoplace no)
@@
 				(path "/d0a98fce-b133-4503-8f8a-83b2a1eed591/7b29c749-8ab5-43b5-aee9-52b112811e58"
 					(reference "#PWR0869997685")
+					(unit 1)
+				)
+			)
+		)
+	)
+	(symbol
+		(lib_id "power:+5V")
+		(at 48.26 72.39 0)
+		(unit 1)
+		(body_style 1)
+		(exclude_from_sim no)
+		(in_bom yes)
+		(on_board yes)
+		(in_pos_files yes)
+		(dnp no)
+		(fields_autoplaced yes)
+		(property "Reference" "#PWR021"
+			(at 48.26 76.2 0)
+			(hide yes)
+			(show_name no)
+			(do_not_autoplace no)
+			(effects
+				(font
+					(size 1.27 1.27)
+				)
+			)
+		)
+		(property "Value" "+3V3"
+			(at 48.26 68.8881 0)
+			(show_name no)
+			(do_not_autoplace no)
+			(effects
+				(font
+					(size 1.27 1.27)
+				)
+			)
+		)
+		(property "Footprint" ""
+			(at 48.26 72.39 0)
+			(hide yes)
+			(show_name no)
+			(do_not_autoplace no)
+			(effects
+				(font
+					(size 1.27 1.27)
+				)
+			)
+		)
+		(property "Datasheet" ""
+			(at 48.26 72.39 0)
+			(hide yes)
+			(show_name no)
+			(do_not_autoplace no)
+			(effects
+				(font
+					(size 1.27 1.27)
+				)
+			)
+		)
+		(property "Description" ""
+			(at 48.26 72.39 0)
+			(show_name no)
+			(do_not_autoplace no)
+			(effects
+				(font
+					(size 1.27 1.27)
+				)
+			)
+		)
+		(pin "1"
+		)
+		(instances
+			(project "blackpants"
+				(path "/d0a98fce-b133-4503-8f8a-83b2a1eed591/7b29c749-8ab5-43b5-aee9-52b112811e58"
+					(reference "#PWR021")
 					(unit 1)
 				)
@@
 	)
 	(symbol
-		(lib_id "A523Power:VCC_PG")
-		(at 182.88 35.56 0)
-		(unit 1)
-		(body_style 1)
-		(exclude_from_sim no)
-		(in_bom no)
-		(on_board yes)
-		(in_pos_files yes)
-		(dnp no)
-		(property "Reference" "#PWR0465010071"
-			(at 182.88 35.56 0)
-			(hide yes)
-			(show_name no)
-			(do_not_autoplace no)
-			(effects
-				(font
-					(size 1.016 1.016)
-				)
-			)
-		)
-		(property "Value" "VCC_PG"
-			(at 182.88 31.75 0)
-			(show_name no)
-			(do_not_autoplace no)
-			(effects
-				(font
-					(size 1.016 1.016)
-				)
-			)
-		)
-		(property "Footprint" ""
-			(at 182.88 35.56 0)
-			(show_name no)
-			(do_not_autoplace no)
-			(effects
-				(font
-					(size 1.27 1.27)
-				)
-			)
-		)
-		(property "Datasheet" ""
-			(at 182.88 35.56 0)
-			(show_name no)
-			(do_not_autoplace no)
-			(effects
-				(font
-					(size 1.27 1.27)
-				)
-			)
-		)
-		(property "Description" ""
-			(at 182.88 35.56 0)
-			(show_name no)
-			(do_not_autoplace no)
-			(effects
-				(font
-					(size 1.27 1.27)
-				)
-			)
-		)
-		(pin "1"
-		)
-		(instances
-			(project "blackpants"
-				(path "/d0a98fce-b133-4503-8f8a-83b2a1eed591/7b29c749-8ab5-43b5-aee9-52b112811e58"
-					(reference "#PWR0465010071")
-					(unit 1)
-				)
-			)
-		)
-	)
-	(symbol
 		(lib_id "A523Power:VCC_3V3")
 		(at 165.1 62.23 0)
@@
 					(unit 1)
 				)
+			)
+		)
+	)
+	(symbol
+		(lib_id "power:+5V")
+		(at 33.02 80.01 0)
+		(unit 1)
+		(body_style 1)
+		(exclude_from_sim no)
+		(in_bom yes)
+		(on_board yes)
+		(in_pos_files yes)
+		(dnp no)
+		(fields_autoplaced yes)
+		(property "Reference" "#PWR020"
+			(at 33.02 83.82 0)
+			(hide yes)
+			(show_name no)
+			(do_not_autoplace no)
+			(effects
+				(font
+					(size 1.27 1.27)
+				)
+			)
+		)
+		(property "Value" "+3V3"
+			(at 33.02 76.5081 0)
+			(show_name no)
+			(do_not_autoplace no)
+			(effects
+				(font
+					(size 1.27 1.27)
+				)
+			)
+		)
+		(property "Footprint" ""
+			(at 33.02 80.01 0)
+			(hide yes)
+			(show_name no)
+			(do_not_autoplace no)
+			(effects
+				(font
+					(size 1.27 1.27)
+				)
+			)
+		)
+		(property "Datasheet" ""
+			(at 33.02 80.01 0)
+			(hide yes)
+			(show_name no)
+			(do_not_autoplace no)
+			(effects
+				(font
+					(size 1.27 1.27)
+				)
+			)
+		)
+		(property "Description" ""
+			(at 33.02 80.01 0)
+			(show_name no)
+			(do_not_autoplace no)
+			(effects
+				(font
+					(size 1.27 1.27)
+				)
+			)
+		)
+		(pin "1"
+		)
+		(instances
+			(project "blackpants"
+				(path "/d0a98fce-b133-4503-8f8a-83b2a1eed591/7b29c749-8ab5-43b5-aee9-52b112811e58"
+					(reference "#PWR020")
+					(unit 1)
+				)
