File: ee/integrated/blackpants.kicad_pcb (KiCad board)
At the start: 6 copper layers, 90 x 153 mm, 313 parts, among them J101 USB-C / recovery, J105 microSD / boot, J3 Conn_ARM_SWD_TagConnect_TC203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, J4 USB_A, J5 USB_A, J701 Antenna, J8 USB-C / charge + keyboard, J801 Conn_01x20_MountingPin, SW1 SW_Push, SW101 FEL, U1 STM32F042C6Ux, U101 USBLC6-2SC6, U11 TPSGM7227YUWQ10G, U12 USBLC6-2SC6, U15 AP3032, U201 A523, U3 USB2514B_Bi, U301 NT6AN512T32AV-J2, U4 MIC2026-1xM, U5 USBLC6-2SC6, U501 AXP717C, U502 AXP323, U6 USBLC6-2SC6, U7 AOZ1280CI, U701 RTL8723DS, U801 AP3036B, U901 TPS61230DRCR, Y1 24Mhz, Y201 24MHz / CL20pF / 20ppm, Y202 32.768kHz / CL12.5pF / 20ppm

Commit message: Worked on the layout.
Parts:
- removed C252, C253: 22pF, Capacitor_SMD:C_0402_1005Metric
- removed C282: 10uF, Capacitor_SMD:C_0402_1005Metric
- removed C523, C524, C527, C529, C530, C532, C534: 2.2uF, Capacitor_SMD:C_0402_1005Metric
- removed JP801: SolderJumper_2_Bridged, Jumper:SolderJumper-2_P1.3mm_Bridged_Pad1.0x1.5mm
- removed R202: 10M, Resistor_SMD:R_0402_1005Metric
- removed Y202: 32.768kHz / CL12.5pF / 20ppm, Crystal:Crystal_SMD_3215-2Pin_3.2x1.5mm
- C258, C260: moved to B.Cu
- moved C258 44.4 mm to (112.1, 68.0)
- moved C260 13.8 mm to (48.9, 70.9), turned to 90 degrees
- moved H1 12.0 mm to (33.0, 30.0)
Connections:
- C265 pad 1: VCC_PE -> +3V3
- C266 pad 1: VCC_PG -> +3V3
- C705 pad 1: VCC_PG -> +3V3
- J801 pad 14: Net-(J801-Pin_14) -> +3V3
- R710 pad 1: VCC_PG -> +3V3
- R711 pad 1: VCC_PG -> +3V3
- R712 pad 1: VCC_PG -> +3V3
- R713 pad 1: VCC_PG -> +3V3
- R714 pad 1: VCC_PG -> +3V3
- R715 pad 1: VCC_PG -> +3V3
- U201 pad A10: /BT_WAKE -> /BT_HOST_WAKE
- U201 pad AH11: /A523 Clocks/X32KOUT -> unconnected-(U201C-X32KOUT-PadAH11)
- U201 pad AH12: /A523 Clocks/X32KIN -> unconnected-(U201C-X32KIN-PadAH12)
- U201 pad J6: VCC_PE -> +3V3
- U201 pad N6: VCC_PG -> +3V3
- U501 pad 13: ALDO1_UNUSED -> unconnected-(U501C-ALDO1-Pad13)
- U501 pad 14: VCC_PE -> unconnected-(U501C-ALDO2-Pad14)
- U501 pad 18: VCC_PG -> unconnected-(U501C-BLDO1-Pad18)
- U501 pad 21: BLDO3_UNUSED -> unconnected-(U501C-BLDO3-Pad21)
- U501 pad 22: BLDO4_UNUSED -> unconnected-(U501C-BLDO4-Pad22)
- U501 pad 24: CLDO2_UNUSED -> unconnected-(U501C-CLDO2-Pad24)
- U501 pad 27: VCC_LCD -> unconnected-(U501C-CLDO4-Pad27)
- U701 pad 22: VCC_PG -> +3V3
- U701 pad 7: /BT_WAKE -> /BT_HOST_WAKE
Routing:
- net VCC_PG: track 93.5 -> 0.00 mm, vias 8 -> 0
- net +3V3: track 280.0 -> 351.6 mm, vias 31 -> 42
- net (no net): track 98.8 -> 36.0 mm, vias 11 -> 4
- net VCC_3V3: track 200.1 -> 164.4 mm, vias 26 -> 22
- net /BT_WAKE: track 43.9 -> 15.5 mm, vias 5 -> 1
- net VCC_1V8: track 88.8 -> 60.5 mm, vias 13 -> 8
- net VDD_CPUS: track 42.5 -> 22.4 mm, vias 8 -> 5
- net VCC_PE: track 15.0 -> 0.00 mm, vias 4 -> 0
- net /AP_NMI: track 60.0 -> 74.8 mm
- net /FEL_N: track 34.2 -> 20.8 mm, vias 4 -> 1
- net ALDO1_UNUSED: track 9.63 -> 0.00 mm, vias 1 -> 0
- net GND: track 167.9 -> 158.5 mm, vias 458 -> 445
- net unconnected-(U501C-BLDO3-Pad21): track 0.00 -> 8.99 mm, vias 0 -> 2
- net BLDO3_UNUSED: track 8.99 -> 0.00 mm, vias 2 -> 0
- net /UART0_RX: track 52.9 -> 44.2 mm
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- removed copper zone on F.Cu, net VDD_DNR
Other:
- board text added: "HIGH SPEED"
- board text added: "LEFT <-> RIGHT"
- board text added: "Power"
- board text added: "SIGNAL"
- board text added: "UP <-> DOWN"
