File: ee/integrated/dsi.kicad_sch (KiCad schematic)
At the start: 8 parts, among them J801 Conn_01x20_MountingPin, U801 AP3036B

Commit message: Added a523 components.
Connections:
- net CLKN renamed DSI_CKN
- net CLKP renamed DSI_CKP
- net D0N renamed DSI_D0N
- net D0P renamed DSI_D0P
- net D1N renamed DSI_D1N
- net D1P renamed DSI_D1P
- net LCD_DIM renamed LCD_PWM

Commit message: Working on the schematic.
Connections:
- net DSI_CKN renamed DSI.CKN
- net DSI_CKP renamed DSI.CKP
- net DSI_D0N renamed DSI.D0N
- net DSI_D0P renamed DSI.D0P
- net DSI_D1N renamed DSI.D1N
- net DSI_D1P renamed DSI.D1P
Other:
- note removed: "Both are bottom contacts."
Changed lines of the file:
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@@
 	(generator_version "10.0")
 	(paper "A4")
-	(text "Both are bottom contacts."
-		(exclude_from_sim no)
-		(at 139.954 106.426 0)
-		(effects
-			(font
-				(size 1.27 1.27)
-			)
-		)
-	)
 	(text "On panel"
 		(exclude_from_sim no)
@@
 		(at 175.26 88.9)
 	)
+	(bus_entry
+		(at 129.54 111.76)
+		(size 2.54 2.54)
+		(stroke
+			(width 0)
+			(type default)
+		)
+	)
+	(bus_entry
+		(at 129.54 116.84)
+		(size 2.54 2.54)
+		(stroke
+			(width 0)
+			(type default)
+		)
+	)
+	(bus_entry
+		(at 129.54 109.22)
+		(size 2.54 2.54)
+		(stroke
+			(width 0)
+			(type default)
+		)
+	)
+	(bus_entry
+		(at 129.54 101.6)
+		(size 2.54 2.54)
+		(stroke
+			(width 0)
+			(type default)
+		)
+	)
+	(bus_entry
+		(at 129.54 104.14)
+		(size 2.54 2.54)
+		(stroke
+			(width 0)
+			(type default)
+		)
+	)
+	(bus_entry
+		(at 129.54 119.38)
+		(size 2.54 2.54)
+		(stroke
+			(width 0)
+			(type default)
+		)
+	)
 	(wire
 		(pts
@@
 	(wire
 		(pts
-			(xy 163.83 121.92) (xy 175.26 121.92)
-		)
-		(stroke
-			(width 0)
-			(type default)
-		)
-	)
-	(wire
-		(pts
 			(xy 172.72 91.44) (xy 175.26 91.44)
 		)
@@
 	(wire
 		(pts
+			(xy 132.08 121.92) (xy 175.26 121.92)
+		)
+		(stroke
+			(width 0)
+			(type default)
+		)
+	)
+	(wire
+		(pts
 			(xy 142.24 63.5) (xy 142.24 66.04)
 		)
@@
 	(wire
 		(pts
-			(xy 163.83 114.3) (xy 175.26 114.3)
-		)
-		(stroke
-			(width 0)
-			(type default)
-		)
-	)
-	(wire
-		(pts
-			(xy 163.83 104.14) (xy 175.26 104.14)
-		)
-		(stroke
-			(width 0)
-			(type default)
-		)
-	)
-	(wire
-		(pts
 			(xy 165.1 124.46) (xy 165.1 127)
 		)
@@
 	(wire
 		(pts
+			(xy 132.08 111.76) (xy 175.26 111.76)
+		)
+		(stroke
+			(width 0)
+			(type default)
+		)
+	)
+	(wire
+		(pts
 			(xy 165.1 101.6) (xy 165.1 109.22)
 		)
@@
 	(wire
 		(pts
-			(xy 163.83 106.68) (xy 175.26 106.68)
+			(xy 132.08 119.38) (xy 175.26 119.38)
 		)
 		(stroke
@@
 		)
 	)
+	(bus
+		(pts
+			(xy 123.19 95.25) (xy 129.54 95.25)
+		)
+		(stroke
+			(width 0)
+			(type default)
+		)
+	)
 	(wire
 		(pts
@@
 		)
 	)
-	(wire
-		(pts
-			(xy 163.83 111.76) (xy 175.26 111.76)
+	(bus
+		(pts
+			(xy 129.54 95.25) (xy 129.54 119.38)
 		)
 		(stroke
@@
 		)
 	)
+	(wire
+		(pts
+			(xy 132.08 104.14) (xy 175.26 104.14)
+		)
+		(stroke
+			(width 0)
+			(type default)
+		)
+	)
 	(polyline
 		(pts
@@
 	(wire
 		(pts
-			(xy 163.83 119.38) (xy 175.26 119.38)
-		)
-		(stroke
-			(width 0)
-			(type default)
-		)
-	)
-	(wire
-		(pts
 			(xy 144.78 38.1) (xy 144.78 41.91)
 		)
@@
 	(wire
 		(pts
+			(xy 132.08 114.3) (xy 175.26 114.3)
+		)
+		(stroke
+			(width 0)
+			(type default)
+		)
+	)
+	(wire
+		(pts
 			(xy 120.65 43.18) (xy 120.65 45.72)
 		)
@@
 	(wire
 		(pts
+			(xy 132.08 106.68) (xy 175.26 106.68)
+		)
+		(stroke
+			(width 0)
+			(type default)
+		)
+	)
+	(wire
+		(pts
 			(xy 120.65 43.18) (xy 124.46 43.18)
 		)
@@
 			(width 0)
 			(type default)
+		)
+	)
+	(label "DSI.CKP"
+		(at 151.13 111.76 180)
+		(effects
+			(font
+				(size 1.27 1.27)
+			)
+			(justify right bottom)
 		)
 	)
@@
 		)
 	)
+	(label "DSI.D1P"
+		(at 151.13 104.14 180)
+		(effects
+			(font
+				(size 1.27 1.27)
+			)
+			(justify right bottom)
+		)
+	)
 	(label "LED_K"
 		(at 171.45 81.28 180)
@@
 		)
 	)
+	(label "DSI.D0P"
+		(at 151.13 119.38 180)
+		(effects
+			(font
+				(size 1.27 1.27)
+			)
+			(justify right bottom)
+		)
+	)
 	(label "LED_A"
 		(at 144.78 38.1 0)
@@
 		)
 	)
-	(hierarchical_label "DSI_D0N"
-		(shape bidirectional)
-		(at 163.83 121.92 180)
-		(effects
-			(font
-				(size 1.27 1.27)
-			)
-			(justify right)
+	(label "DSI.D0N"
+		(at 151.13 121.92 180)
+		(effects
+			(font
+				(size 1.27 1.27)
+			)
+			(justify right bottom)
+		)
+	)
+	(label "DSI.CKN"
+		(at 151.13 114.3 180)
+		(effects
+			(font
+				(size 1.27 1.27)
+			)
+			(justify right bottom)
+		)
+	)
+	(label "DSI.D1N"
+		(at 151.13 106.68 180)
+		(effects
+			(font
+				(size 1.27 1.27)
+			)
+			(justify right bottom)
 		)
 	)
@@
 		)
 	)
-	(hierarchical_label "DSI_CKN"
-		(shape bidirectional)
-		(at 163.83 114.3 180)
-		(effects
-			(font
-				(size 1.27 1.27)
-			)
-			(justify right)
-		)
-	)
 	(hierarchical_label "LCD_TE"
 		(shape input)
@@
 		)
 	)
-	(hierarchical_label "DSI_D1P"
+	(hierarchical_label "DSI{DSI}"
 		(shape bidirectional)
-		(at 163.83 104.14 180)
-		(effects
-			(font
-				(size 1.27 1.27)
-			)
-			(justify right)
-		)
-	)
-	(hierarchical_label "DSI_D0P"
-		(shape bidirectional)
-		(at 163.83 119.38 180)
-		(effects
-			(font
-				(size 1.27 1.27)
-			)
-			(justify right)
-		)
-	)
-	(hierarchical_label "DSI_CKP"
-		(shape bidirectional)
-		(at 163.83 111.76 180)
-		(effects
-			(font
-				(size 1.27 1.27)
-			)
-			(justify right)
-		)
-	)
-	(hierarchical_label "DSI_D1N"
-		(shape bidirectional)
-		(at 163.83 106.68 180)
-		(effects
-			(font
+		(at 123.19 95.25 180)
+		(effects
+			(font

Commit message: Worked on the layout.
Parts:
- removed JP801: SolderJumper_2_Bridged, Jumper:SolderJumper-2_P1.3mm_Bridged_Pad1.0x1.5mm, symbol Jumper:SolderJumper_2_Bridged
Connections:
- net +3V3: now also J801.14 (Pin_14)
Changed lines of the file:
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@@
 	)
 	(junction
-		(at 161.29 90.17)
+		(at 161.29 91.44)
 		(diameter 0)
 		(color 0 0 0 0)
@@
 	(wire
 		(pts
-			(xy 163.83 93.98) (xy 161.29 93.98)
-		)
-		(stroke
-			(width 0)
-			(type default)
-		)
-	)
-	(wire
-		(pts
-			(xy 172.72 91.44) (xy 175.26 91.44)
+			(xy 161.29 93.98) (xy 175.26 93.98)
 		)
 		(stroke
@@
 	(wire
 		(pts
-			(xy 175.26 93.98) (xy 171.45 93.98)
-		)
-		(stroke
-			(width 0)
-			(type default)
-		)
-	)
-	(wire
-		(pts
 			(xy 111.76 57.15) (xy 132.08 57.15)
 		)
@@
 	(wire
 		(pts
+			(xy 161.29 87.63) (xy 161.29 93.98)
+		)
+		(stroke
+			(width 0)
+			(type default)
+		)
+	)
+	(wire
+		(pts
 			(xy 171.45 81.28) (xy 175.26 81.28)
 		)
@@
 	(wire
 		(pts
-			(xy 172.72 90.17) (xy 161.29 90.17)
+			(xy 161.29 91.44) (xy 175.26 91.44)
 		)
 		(stroke
@@
 	(wire
 		(pts
-			(xy 161.29 90.17) (xy 161.29 93.98)
-		)
-		(stroke
-			(width 0)
-			(type default)
-		)
-	)
-	(wire
-		(pts
-			(xy 172.72 90.17) (xy 172.72 91.44)
-		)
-		(stroke
-			(width 0)
-			(type default)
-		)
-	)
-	(wire
-		(pts
 			(xy 154.94 55.88) (xy 154.94 58.42)
 		)
@@
 		(pts
 			(xy 138.43 43.18) (xy 138.43 44.45)
-		)
-		(stroke
-			(width 0)
-			(type default)
-		)
-	)
-	(wire
-		(pts
-			(xy 161.29 87.63) (xy 161.29 90.17)
 		)
 		(stroke
@@
 					(unit 1)
 				)
-			)
-		)
-	)
-	(symbol
-		(lib_id "Jumper:SolderJumper_2_Bridged")
-		(at 167.64 93.98 0)
-		(unit 1)
-		(body_style 1)
-		(exclude_from_sim yes)
-		(in_bom no)
-		(on_board yes)
-		(in_pos_files yes)
-		(dnp no)
-		(property "Reference" "JP801"
-			(at 167.64 92.202 0)
-			(show_name no)
-			(do_not_autoplace no)
-			(effects
-				(font
-					(size 1.27 1.27)
-				)
-			)
-		)
-		(property "Value" "SolderJumper_2_Bridged"
-			(at 167.64 90.17 0)
-			(hide yes)
-			(show_name no)
-			(do_not_autoplace no)
-			(effects
-				(font
-					(size 1.27 1.27)
-				)
-			)
-		)
-		(property "Footprint" "Jumper:SolderJumper-2_P1.3mm_Bridged_Pad1.0x1.5mm"
-			(at 167.64 93.98 0)
-			(hide yes)
-			(show_name no)
-			(do_not_autoplace no)
-			(effects
-				(font
-					(size 1.27 1.27)
-				)
-			)
-		)
-		(property "Datasheet" ""
-			(at 167.64 93.98 0)
-			(hide yes)
-			(show_name no)
-			(do_not_autoplace no)
-			(effects
-				(font
-					(size 1.27 1.27)
-				)
-			)
-		)
-		(property "Description" "Solder Jumper, 2-pole, closed/bridged"
-			(at 167.64 93.98 0)
-			(hide yes)
-			(show_name no)
-			(do_not_autoplace no)
-			(effects
-				(font
-					(size 1.27 1.27)
-				)
-			)
-		)
-		(pin "2"
-		)
-		(pin "1"
-		)
-		(instances
-			(project "blackpants"
-				(path "/d0a98fce-b133-4503-8f8a-83b2a1eed591/4c080231-9d8c-4e1e-a878-bc11551bd68a"
-					(reference "JP801")
-					(unit 1)
-				)
