File: ee/integrated/peripheral_power.kicad_sch (KiCad schematic)
At the start: 18 parts, among them U7 AOZ1280CI, U901 TPS61230DRCR

Commit message: Working on the schematic.
Other:
- moved on the sheet: C911, R910, R911

Commit message: Worked on the layout.
Changed lines of the file:
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@@
 	(wire
 		(pts
+			(xy 46.99 41.91) (xy 46.99 45.72)
+		)
+		(stroke
+			(width 0)
+			(type default)
+		)
+	)
+	(wire
+		(pts
 			(xy 35.56 139.7) (xy 35.56 140.97)
 		)
@@
 	(wire
 		(pts
-			(xy 71.12 45.72) (xy 45.72 45.72)
+			(xy 46.99 45.72) (xy 71.12 45.72)
 		)
 		(stroke
@@
 	(symbol
 		(lib_id "A523Power:VSYS")
-		(at 45.72 45.72 0)
+		(at 46.99 41.91 0)
 		(unit 1)
 		(body_style 1)
@@
 		(dnp no)
 		(property "Reference" "#PWR0624090499"
-			(at 45.72 45.72 0)
+			(at 46.99 41.91 0)
 			(hide yes)
 			(show_name no)
@@
 		)
 		(property "Value" "VSYS"
-			(at 45.72 41.91 0)
+			(at 46.99 38.1 0)
 			(show_name no)
 			(do_not_autoplace no)
@@
 		)
 		(property "Footprint" ""
-			(at 45.72 45.72 0)
+			(at 46.99 41.91 0)
 			(show_name no)
 			(do_not_autoplace no)
@@
 		)
 		(property "Datasheet" ""
-			(at 45.72 45.72 0)
+			(at 46.99 41.91 0)
 			(show_name no)
 			(do_not_autoplace no)
@@
 		)
 		(property "Description" ""
-			(at 45.72 45.72 0)
+			(at 46.99 41.91 0)
 			(show_name no)
 			(do_not_autoplace no)
