File: ee/integrated/wifi.kicad_sch (KiCad schematic)
At the start: 20 parts, among them J701 Conn_Coaxial, U701 RTL8723DS

Commit message: Added a523 components.
Parts:
- removed C706, C707: 10uF, Capacitor_SMD:C_0603_1608Metric, symbol Device:C_Small
- removed R701: 10K, Resistor_SMD:R_0402_1005Metric, symbol Device:R_Small_US
- removed R702, R705: 1k, Resistor_SMD:R_0402_1005Metric, symbol Device:R_Small_US
- removed R703, R708: 0R, Resistor_SMD:R_0402_1005Metric, symbol Device:R_Small_US
- removed R704: 100K, Resistor_SMD:R_0402_1005Metric, symbol Device:R_Small_US
- removed R706: 100k, Resistor_SMD:R_0402_1005Metric, symbol Device:R_Small_US
- removed R707: 10k, Resistor_SMD:R_0402_1005Metric, symbol Device:R_Small_US
- removed RN701, RN702: 10k, Resistor_SMD:R_Array_Convex_4x0402, symbol Device:R_Pack04
- added R703: 0, Resistor_SMD:R_0402_1005Metric, symbol Device:R_Small
- added R710, R711, R712, R713, R714: 10k, Resistor_SMD:R_0201_0603Metric, symbol Device:R_Small
- added R715: 10k, Resistor_SMD:R_0402_1005Metric, symbol Device:R_Small
- added R716, R717, R718: 100k, Resistor_SMD:R_0402_1005Metric, symbol Device:R_Small
- C701, C702: value NC -> DNP; Dielectric (none) -> X5R/X7R; Voltage (none) -> 10V; now in the parts list
- C703: Dielectric (none) -> X5R/X7R; MPN LMK107BBJ106MALT -> (none); Voltage (none) -> 10V
- C704: value NC -> 100nF; Dielectric (none) -> X5R/X7R; Voltage (none) -> 10V; now fitted; now in the parts list
- C705: value 10uF -> 100nF; footprint Capacitor_SMD:C_0603_1608Metric -> Capacitor_SMD:C_0402_1005Metric; Dielectric (none) -> X5R/X7R; MPN LMK107BBJ106MALT -> (none); Voltage (none) -> 10V
- J701: value Conn_Coaxial -> Antenna; MPN SMA-KWE901 -> (none)
- L701: value 120R@100MHz -> 120R @100MHz / >=0.6A; MPN BLM18KG121TN1D -> (none)
- U701: MPN RTL8723DS -> (none)
Connections:
- net GND: now also R716.2, R717.2, R718.2
- net WL_REG_ON: now also R716.1
- net BT_RXD: now reaches U701.43 (UART_RXD)
- net at J701.1 (In): now also C702.1, R703.2; no longer C701.1
- net BT_TXD: now reaches U701.42 (UART_TXD)
- net RF_ANT: now reaches U701.2 (WIFI/BT_ANT)
- net RF_ANT: now also C701.1, R703.1; no longer C702.1
- net +3.3VA renamed VCC_WIFI
- net VCC_WIFI: now also C704.1; no longer C705.1, U701.22 (VDD_IO)
- net CTS_N renamed BT_RTS_N
- net HOST_WAKE renamed BT_HOST_WAKE
- net LPO renamed CLK32K
- net CLK32K: now also R715.2
- net RST_N renamed BT_RESET_N
- net BT_RESET_N: now also R717.1; no longer C704.1
- net RTS_N renamed BT_CTS_N
- net SDC1.CLK renamed SD1_CLK
- net SDC1.CMD renamed SD1_CMD
- net SD1_CMD: now also R710.2
- net SDC1.D0 renamed SD1_D0
- net SD1_D0: now also R711.2
- net SDC1.D1 renamed SD1_D1
- net SD1_D1: now also R712.2
- net SDC1.D2 renamed SD1_D2
- net SD1_D2: now also R713.2
- net SDC1.D3 renamed SD1_D3
- net SD1_D3: now also R714.2
- net WAKE renamed BT_WAKE
- net BT_WAKE: now also R718.1
- new net VCC_PG: C705.1, R710.1, R711.1, R712.1, R713.1, R714.1, R715.1, U701.22 (VDD_IO)
- no-connect marks 18 -> 19
Other:
- note added: "Program BLDO1 = 3.3V before enabling PG / PH outputs. VBAT is filtered +3V3; VDD_IO is the separately sequenced VCC_PG. Module TX/RTS -> SoC RX/CTS; module RX/CTS <- SoC TX/RTS. X32KFOUT is open drain; R715 pulls it up to VCC_PG."
- note removed: "50Ω"
- note removed: "?"
- note removed: "A"
- note removed: "B"
- note removed: "C"
- note removed: "Check L5 package and PN it was MMZ2012R121AT000 before"
- note removed: "D"
- note removed: "RTL8723DS - Populate B and D XR829 - Populate A and C"
- title: (none) -> RTL8723DS Wi-Fi and Bluetooth

Commit message: Working on the schematic.
Connections:
- net BT_CTS_N renamed BT.~{RTS}
- net BT_RTS_N renamed BT.~{CTS}
- net BT_RXD renamed BT.TX
- net BT_TXD renamed BT.RX
- net SD1_CLK renamed SD1.CLK
- net SD1_CMD renamed SD1.CMD
- net SD1_D0 renamed SD1.D0
- net SD1_D1 renamed SD1.D1
- net SD1_D2 renamed SD1.D2
- net SD1_D3 renamed SD1.D3

Commit message: Removed USB sheets and moved the parts to the main sheets.
Connections:
- net CLK32K: no longer U701.24 (LPO)
Changed lines of the file:
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@@
-	(wire
-		(pts
-			(xy 81.28 99.06) (xy 76.2 99.06)
-		)
-		(stroke
-			(width 0)
-			(type default)
-		)
-	)
 	(wire
 		(pts
@@
 		(effects
 			(font
-				(size 1.27 1.27)
-			)
-			(justify right)
-		)
-	)
-	(hierarchical_label "CLK32K"
-		(shape bidirectional)
-		(at 76.2 99.06 180)
-		(effects
-			(font

Commit message: Worked on the layout.
Connections:
- net VCC_PG is gone; now on net +3V3: C705.1, R710.1, R711.1, R712.1, R713.1, R714.1, R715.1, U701.22 (VDD_IO)
